Commit message: Retune linear elevator's controller, remove velocity multiplier from interface and fix co2 plugin's message.

File: pandora_gazebo_description/urdf/gears/sdf_configurations.xacro (robot description, xacro)
@@ -39,5 +39,5 @@
     <xacro:property name="enable_wheel_joint_physics" value="false" />
     <!-- ================================================================== -->
-    <xacro:property name="enable_linear_elevator_joint_physics" value="false" /> <!-- FIXME -->
+    <xacro:property name="enable_linear_elevator_joint_physics" value="true" />
     <!-- ================================================================== -->
     <xacro:property name="enable_linear_head_pitch_joint_physics" value="false" />
