Commit message: Adjust linear's limits and reduce wheels' stiffness.

File: pandora_gazebo_description/urdf/gears/gears_simplified.gazebo.xacro (robot description, xacro)
@@ -25,5 +25,5 @@
   <xacro:property name="wheel_mu_1" value="0.675" />
   <xacro:property name="wheel_mu_2" value="0.675" />
-  <xacro:property name="wheel_k_p" value="10000000.0" />
+  <xacro:property name="wheel_k_p" value="1000000.0" />
   <xacro:property name="wheel_k_d" value="0.8" />
   <xacro:property name="wheel_min_depth" value="0.001" />

File: pandora_gazebo_description/urdf/gears/sdf_configurations.xacro (robot description, xacro)
@@ -67,5 +67,5 @@
   <xacro:property name="wheel_mu_1" value="0.675" />
   <xacro:property name="wheel_mu_2" value="0.675" />
-  <xacro:property name="wheel_k_p" value="10000000.0" />
+  <xacro:property name="wheel_k_p" value="1000000.0" />
   <xacro:property name="wheel_k_d" value="0.8" />
   <xacro:property name="wheel_min_depth" value="0.001" />

Commit message: Adjust physics.

File: pandora_gazebo_description/urdf/gears/gears_simplified.gazebo.xacro (robot description, xacro)
@@ -23,9 +23,9 @@
   <!-- XXX: Get from config -->
   <xacro:property name="robot_namespace" value="" />
-  <xacro:property name="wheel_mu_1" value="0.675" />
-  <xacro:property name="wheel_mu_2" value="0.675" />
-  <xacro:property name="wheel_k_p" value="1000000.0" />
+  <xacro:property name="wheel_mu_1" value="0.65" />
+  <xacro:property name="wheel_mu_2" value="0.65" />
+  <xacro:property name="wheel_k_p" value="100000000.0" />
   <xacro:property name="wheel_k_d" value="0.8" />
-  <xacro:property name="wheel_min_depth" value="0.001" />
+  <xacro:property name="wheel_min_depth" value="0.00001" />
   <xacro:property name="wheel_max_contacts" value="1" />
 <!-- Load URDF ############################################################ -->

File: pandora_gazebo_description/urdf/gears/sdf_configurations.xacro (robot description, xacro)
@@ -65,9 +65,9 @@
 <!-- Joint Physics ######################################################## -->
   <!-- Wheels ============================================================= -->
-  <xacro:property name="wheel_mu_1" value="0.675" />
-  <xacro:property name="wheel_mu_2" value="0.675" />
-  <xacro:property name="wheel_k_p" value="1000000.0" />
+  <xacro:property name="wheel_mu_1" value="0.65" />
+  <xacro:property name="wheel_mu_2" value="0.65" />
+  <xacro:property name="wheel_k_p" value="100000000.0" />
   <xacro:property name="wheel_k_d" value="0.8" />
-  <xacro:property name="wheel_min_depth" value="0.001" />
+  <xacro:property name="wheel_min_depth" value="0.00001" />
   <xacro:property name="wheel_max_contacts" value="1" />
   <!-- ==================================================================== -->

Commit message: Adjust physics and add camera sensor.

File: pandora_gazebo_description/urdf/gears/gears_simplified.gazebo.xacro (robot description, xacro)
@@ -23,9 +23,9 @@
   <!-- XXX: Get from config -->
   <xacro:property name="robot_namespace" value="" />
-  <xacro:property name="wheel_mu_1" value="0.65" />
-  <xacro:property name="wheel_mu_2" value="0.65" />
-  <xacro:property name="wheel_k_p" value="100000000.0" />
-  <xacro:property name="wheel_k_d" value="0.8" />
-  <xacro:property name="wheel_min_depth" value="0.00001" />
+  <xacro:property name="wheel_mu_1" value="0.45" />
+  <xacro:property name="wheel_mu_2" value="0.45" />
+  <xacro:property name="wheel_k_p" value="10000000.0" />
+  <xacro:property name="wheel_k_d" value="1.0" />
+  <xacro:property name="wheel_min_depth" value="0.0001" />
   <xacro:property name="wheel_max_contacts" value="1" />
 <!-- Load URDF ############################################################ -->

Commit message: Revert physics changes.

File: pandora_gazebo_description/urdf/gears/gears_simplified.gazebo.xacro (robot description, xacro)
@@ -24,9 +24,9 @@
   <!-- XXX: Get from config -->
   <xacro:property name="robot_namespace" value="" />
-  <xacro:property name="wheel_mu_1" value="0.45" />
-  <xacro:property name="wheel_mu_2" value="0.45" />
-  <xacro:property name="wheel_k_p" value="10000000.0" />
-  <xacro:property name="wheel_k_d" value="1.0" />
-  <xacro:property name="wheel_min_depth" value="0.0001" />
+  <xacro:property name="wheel_mu_1" value="0.675" />
+  <xacro:property name="wheel_mu_2" value="0.675" />
+  <xacro:property name="wheel_k_p" value="100000000.0" />
+  <xacro:property name="wheel_k_d" value="0.8" />
+  <xacro:property name="wheel_min_depth" value="0.00001" />
   <xacro:property name="wheel_max_contacts" value="1" />
 <!-- Load URDF ############################################################ -->

File: pandora_gazebo_description/urdf/gears/sdf_configurations.xacro (robot description, xacro)
@@ -69,9 +69,9 @@
 <!-- Joint Physics ######################################################## -->
   <!-- Wheels ============================================================= -->
-  <xacro:property name="wheel_mu_1" value="0.45" />
-  <xacro:property name="wheel_mu_2" value="0.45" />
-  <xacro:property name="wheel_k_p" value="10000000.0" />
-  <xacro:property name="wheel_k_d" value="1.0" />
-  <xacro:property name="wheel_min_depth" value="0.0001" />
+  <xacro:property name="wheel_mu_1" value="0.675" />
+  <xacro:property name="wheel_mu_2" value="0.675" />
+  <xacro:property name="wheel_k_p" value="100000000.0" />
+  <xacro:property name="wheel_k_d" value="0.8" />
+  <xacro:property name="wheel_min_depth" value="0.00001" />
   <xacro:property name="wheel_max_contacts" value="1" />
   <!-- ==================================================================== -->

Commit message: Adjust downforce on flat surfaces.

File: pandora_gazebo_description/urdf/gears/gears_simplified.gazebo.xacro (robot description, xacro)
@@ -24,8 +24,8 @@
   <!-- XXX: Get from config -->
   <xacro:property name="robot_namespace" value="" />
-  <xacro:property name="wheel_mu_1" value="0.675" />
-  <xacro:property name="wheel_mu_2" value="0.675" />
-  <xacro:property name="wheel_k_p" value="100000000.0" />
-  <xacro:property name="wheel_k_d" value="0.8" />
+  <xacro:property name="wheel_mu_1" value="0.6" />
+  <xacro:property name="wheel_mu_2" value="0.6" />
+  <xacro:property name="wheel_k_p" value="10000000.0" />
+  <xacro:property name="wheel_k_d" value="1.0" />
   <xacro:property name="wheel_min_depth" value="0.00001" />
   <xacro:property name="wheel_max_contacts" value="1" />

Commit message: Refactor latest method.

File: pandora_gazebo_description/urdf/gears/gears_simplified.gazebo.xacro (robot description, xacro)
@@ -28,5 +28,5 @@
   <xacro:property name="wheel_k_p" value="10000000.0" />
   <xacro:property name="wheel_k_d" value="1.0" />
-  <xacro:property name="wheel_min_depth" value="0.00001" />
+  <xacro:property name="wheel_min_depth" value="0.0001" />
   <xacro:property name="wheel_max_contacts" value="1" />
 <!-- Load URDF ############################################################ -->

Commit message: First attemp with low frictions.

File: pandora_gazebo_description/urdf/gears/gears_simplified.gazebo.xacro (robot description, xacro)
@@ -24,6 +24,6 @@
   <!-- XXX: Get from config -->
   <xacro:property name="robot_namespace" value="" />
-  <xacro:property name="wheel_mu_1" value="0.6" />
-  <xacro:property name="wheel_mu_2" value="0.6" />
+  <xacro:property name="wheel_mu_1" value="0.5" />
+  <xacro:property name="wheel_mu_2" value="0.25" />
   <xacro:property name="wheel_k_p" value="10000000.0" />
   <xacro:property name="wheel_k_d" value="1.0" />

File: pandora_gazebo_description/urdf/gears/physics/wheel_link_physics.gazebo.xacro (robot description, xacro)
@@ -19,5 +19,5 @@
       <mu2>${wheel_mu_2}</mu2>
       <!-- ================================================================ -->
-      <!-- <fdir1>1 0 0</fdir1> -->
+      <fdir1>1 0 0</fdir1>
       <!-- ================================================================ -->
       <kp>${wheel_k_p}</kp>

Commit message: Adjust velocity coefficients for new physics.

File: pandora_gazebo_description/urdf/gears/gears_simplified.gazebo.xacro (robot description, xacro)
@@ -24,6 +24,6 @@
   <!-- XXX: Get from config -->
   <xacro:property name="robot_namespace" value="" />
-  <xacro:property name="wheel_mu_1" value="0.5" />
-  <xacro:property name="wheel_mu_2" value="0.25" />
+  <xacro:property name="wheel_mu_1" value="0.6" />
+  <xacro:property name="wheel_mu_2" value="0.3" />
   <xacro:property name="wheel_k_p" value="10000000.0" />
   <xacro:property name="wheel_k_d" value="1.0" />
