Commit message: Finalize description and update all launchers.

File: pandora_gazebo_description/urdf/gears/gears.gazebo.xacro (robot description, xacro)
@@ -4,5 +4,5 @@
 <!-- Import Files ######################################################### -->
   <!-- ==================================================================== -->
-  <xacro:include filename="$(find pandora_robots_description)/urdf/gears/gears.urdf.xacro" /> <!-- FIXME -->
+  <xacro:include filename="$(find pandora_robots_description)/urdf/gears/gears.urdf.xacro" />
   <!-- ==================================================================== -->
   <xacro:include filename="$(find pandora_gazebo_description)/urdf/gears/sdf_configurations.xacro" />
@@ -19,5 +19,5 @@
   <xacro:include filename="$(find pandora_gazebo_description)/urdf/gears/physics/laser_roll_joint_physics.gazebo.xacro" />
   <xacro:include filename="$(find pandora_gazebo_description)/urdf/gears/physics/laser_pitch_joint_physics.gazebo.xacro" />
-  <xacro:include filename="$(find pandora_gazebo_description)/urdf/gears/physics/kinect_head_pitch_joint_physics.gazebo.xacro" />
+  <xacro:include filename="$(find pandora_gazebo_description)/urdf/gears/physics/kinect_pitch_joint_physics.gazebo.xacro" />
   <xacro:include filename="$(find pandora_gazebo_description)/urdf/gears/physics/kinect_yaw_joint_physics.gazebo.xacro" />
   <!-- ==================================================================== -->
@@ -35,10 +35,20 @@
   <xacro:include filename="$(find pandora_gazebo_description)/urdf/gears/transmissions/kinect_sensor_transmission.xacro" />
   <!-- ==================================================================== -->
-  <xacro:include filename="$(find pandora_gazebo_description)/urdf/gears/plugins/pandora_plugin.gazebo.xacro" />
-  <xacro:include filename="$(find pandora_gazebo_description)/urdf/gears/plugins/pandora_plugin.gazebo.xacro" />
-  <xacro:include filename="$(find pandora_gazebo_description)/urdf/gears/plugins/pandora_plugin.gazebo.xacro" />
-  <xacro:include filename="$(find pandora_gazebo_description)/urdf/gears/plugins/ros_plugin.gazebo.xacro" />
-  <xacro:include filename="$(find pandora_gazebo_description)/urdf/gears/plugins/ros_plugin.gazebo.xacro" />
-  <xacro:include filename="$(find pandora_gazebo_description)/urdf/gears/plugins/ros_plugin.gazebo.xacro" />
+  <xacro:include filename="$(find pandora_gazebo_description)/urdf/gears/plugins/pandora_differential_plugin.gazebo.xacro" />
+  <xacro:include filename="$(find pandora_gazebo_description)/urdf/gears/plugins/pandora_p3d_plugin.gazebo.xacro" />
+  <xacro:include filename="$(find pandora_gazebo_description)/urdf/gears/plugins/pandora_imu_stabilizer_plugin.gazebo.xacro" />
+  <xacro:include filename="$(find pandora_gazebo_description)/urdf/gears/plugins/ros_imu_plugin.gazebo.xacro" />
+  <xacro:include filename="$(find pandora_gazebo_description)/urdf/gears/plugins/ros_skid_steer_drive_plugin.gazebo.xacro" />
+  <xacro:include filename="$(find pandora_gazebo_description)/urdf/gears/plugins/ros_control_plugin.gazebo.xacro" />
+  <!-- ==================================================================== -->
+<!-- Load URDF ############################################################ -->
+  <!-- ==================================================================== -->
+  <xacro:if value="$(arg control)" >
+    <xacro:gears_urdf fixed="false" />
+  </xacro:if>
+  <!-- ==================================================================== -->
+  <xacro:unless value="$(arg control)" >
+    <xacro:gears_urdf fixed="true" />
+  </xacro:unless>
   <!-- ==================================================================== -->
 <!-- Load Physics ######################################################### -->
@@ -223,5 +233,5 @@
         <xacro:if value="${enable_laser_sensor}" >
           <xacro:if value="${enable_pandora_imu_stabilizer_plugin}" >
-            <xacro:pandora_imu_stabilizer_plugin />
+            <!-- <xacro:pandora_imu_stabilizer_plugin /> --> <!-- FIXME -->
           </xacro:if>
         </xacro:if>

File: pandora_gazebo_description/urdf/gears/sdf_configurations.xacro (robot description, xacro)
@@ -3,5 +3,5 @@
 <!-- Robot NameSpace ###################################################### -->
   <!-- ==================================================================== -->
-  <xacro:property name="robot_namespace" value="/" />
+  <xacro:property name="robot_namespace" value="" />
   <!-- ==================================================================== -->
 <!-- Elements' Status ##################################################### -->

Commit message: Complete ARM interface.

File: pandora_gazebo_description/urdf/gears/gears.gazebo.xacro (robot description, xacro)
@@ -142,32 +142,102 @@
       <!-- ================================================================ -->
       <xacro:if value="${enable_left_rear_sonar_gazebo_sensor}" >
-        <xacro:sonar_gazebo_sensor name="left_rear" />
+        <xacro:if value="$(arg control)" >
+          <xacro:if value="$(arg interface)" >
+            <xacro:sonar_gazebo_sensor name="left_rear" publish_msg="false" />
+          </xacro:if>
+          <xacro:unless value="$(arg interface)" >
+            <xacro:sonar_gazebo_sensor name="left_rear" publish_msg="true" />
+          </xacro:unless>
+        </xacro:if>
+        <xacro:unless value="$(arg control)" >
+            <xacro:sonar_gazebo_sensor name="left_rear" publish_msg="true" />
+        </xacro:unless>
       </xacro:if>
       <!-- ================================================================ -->
       <xacro:if value="${enable_right_rear_sonar_gazebo_sensor}" >
-        <xacro:sonar_gazebo_sensor name="right_rear" />
-      </xacro:if>
-      <!-- ================================================================ -->
+        <xacro:if value="$(arg control)" >
+          <xacro:if value="$(arg interface)" >
+            <xacro:sonar_gazebo_sensor name="right_rear" publish_msg="false" />
+          </xacro:if>
+          <xacro:unless value="$(arg interface)" >
+            <xacro:sonar_gazebo_sensor name="right_rear" publish_msg="true" />
+          </xacro:unless>
+        </xacro:if>
+        <xacro:unless value="$(arg control)" >
+            <xacro:sonar_gazebo_sensor name="right_rear" publish_msg="true" />
+        </xacro:unless>
+      </xacro:if>
+      <!-- ================================================================ -->
+    </xacro:if>
+    <xacro:if value="${enable_co2_gazebo_sensor}" >
+      <xacro:if value="$(arg control)" >
+        <xacro:if value="$(arg interface)" >
+          <xacro:co2_gazebo_sensor publish_msg="false" />
+        </xacro:if>
+        <xacro:unless value="$(arg interface)" >
+          <xacro:co2_gazebo_sensor publish_msg="true" />
+        </xacro:unless>
+      </xacro:if>
+      <xacro:unless value="$(arg control)" >
+          <xacro:co2_gazebo_sensor publish_msg="true" />
+      </xacro:unless>
     </xacro:if>
     <xacro:if value="${enable_thermal_gazebo_sensors}" >
       <!-- ================================================================ -->
       <xacro:if value="${enable_middle_thermal_gazebo_sensor}" >
-        <xacro:thermal_gazebo_sensor prefix_y="middle" />
+        <xacro:if value="$(arg control)" >
+          <xacro:if value="$(arg interface)" >
+            <xacro:thermal_gazebo_sensor prefix_y="middle" publish_msg="false" />
+          </xacro:if>
+          <xacro:unless value="$(arg interface)" >
+            <xacro:thermal_gazebo_sensor prefix_y="middle" publish_msg="true" />
+          </xacro:unless>
+        </xacro:if>
+        <xacro:unless value="$(arg control)" >
+            <xacro:thermal_gazebo_sensor prefix_y="middle" publish_msg="true" />
+        </xacro:unless>
       </xacro:if>
       <!-- ================================================================ -->
       <xacro:if value="${enable_left_thermal_gazebo_sensor}" >
-        <xacro:thermal_gazebo_sensor prefix_y="left" />
+        <xacro:if value="$(arg control)" >
+          <xacro:if value="$(arg interface)" >
+            <xacro:thermal_gazebo_sensor prefix_y="left" publish_msg="false" />
+          </xacro:if>
+          <xacro:unless value="$(arg interface)" >
+            <xacro:thermal_gazebo_sensor prefix_y="left" publish_msg="true" />
+          </xacro:unless>
+        </xacro:if>
+        <xacro:unless value="$(arg control)" >
+            <xacro:thermal_gazebo_sensor prefix_y="left" publish_msg="true" />
+        </xacro:unless>
       </xacro:if>
       <!-- ================================================================ -->
       <xacro:if value="${enable_right_thermal_gazebo_sensor}" >
-        <xacro:thermal_gazebo_sensor prefix_y="right" />
-      </xacro:if>
-      <!-- ================================================================ -->
-    </xacro:if>
-    <xacro:if value="${enable_co2_gazebo_sensor}" >
-      <xacro:co2_gazebo_sensor />
+        <xacro:if value="$(arg control)" >
+          <xacro:if value="$(arg interface)" >
+            <xacro:thermal_gazebo_sensor prefix_y="right" publish_msg="false" />
+          </xacro:if>
+          <xacro:unless value="$(arg interface)" >
+            <xacro:thermal_gazebo_sensor prefix_y="right" publish_msg="true" />
+          </xacro:unless>
+        </xacro:if>
+        <xacro:unless value="$(arg control)" >
+            <xacro:thermal_gazebo_sensor prefix_y="right" publish_msg="true" />
+        </xacro:unless>
+      </xacro:if>
+      <!-- ================================================================ -->
     </xacro:if>
     <xacro:if value="${enable_microphone_gazebo_sensor}" >
-      <xacro:microphone_gazebo_sensor />
+      <xacro:if value="$(arg control)" >
+        <xacro:if value="$(arg interface)" >
+          <xacro:microphone_gazebo_sensor publish_msg="false" />
+        </xacro:if>
+        <xacro:unless value="$(arg interface)" >
+          <xacro:microphone_gazebo_sensor publish_msg="true" />
+        </xacro:unless>
+      </xacro:if>
+      <xacro:unless value="$(arg control)" >
+          <xacro:microphone_gazebo_sensor publish_msg="true" />
+      </xacro:unless>
     </xacro:if>
   </xacro:if>

File: pandora_gazebo_description/urdf/gears/sensors/co2_sensor.gazebo.xacro (robot description, xacro)
@@ -2,5 +2,6 @@
 <robot xmlns:xacro="http://ros.org/wiki/xacro" >
 <!-- ###################################################################### -->
-  <xacro:macro name="co2_gazebo_sensor" >
+  <xacro:macro name="co2_gazebo_sensor"
+               params="publish_msg" >
     <gazebo reference="co2_link" >
       <sensor name="co2" type="camera" >
@@ -27,4 +28,6 @@
           <topicName>sensors/co2</topicName> <!-- FIXME -->
           <!--============================================================= -->
+          <publishMsg>${publish_msg}</publishMsg>
+          <!--============================================================= -->
         </plugin>
         <!--=============================================================== -->

File: pandora_gazebo_description/urdf/gears/sensors/microphone_sensor.gazebo.xacro (robot description, xacro)
@@ -2,5 +2,6 @@
 <robot xmlns:xacro="http://ros.org/wiki/xacro" >
 <!-- ###################################################################### -->
-  <xacro:macro name="microphone_gazebo_sensor" >
+  <xacro:macro name="microphone_gazebo_sensor"
+               params="publish_msg" >
     <gazebo reference="microphone_link" >
       <sensor name="microphone"
@@ -28,4 +29,6 @@
           <topicName>sensors/sound</topicName> <!-- FIXME -->
           <!--============================================================= -->
+          <publishMsg>${publish_msg}</publishMsg>
+          <!--============================================================= -->
         </plugin>
         <!--=============================================================== -->

File: pandora_gazebo_description/urdf/gears/sensors/sonar_sensor.gazebo.xacro (robot description, xacro)
@@ -3,5 +3,5 @@
 <!-- ###################################################################### -->
   <xacro:macro name="sonar_gazebo_sensor"
-               params="name" >
+               params="name publish_msg" >
     <gazebo reference="${name}_sonar_link" >
       <sensor name="${name}_sonar"
@@ -50,4 +50,6 @@
           <gaussianNoise>0.0</gaussianNoise>
           <!--============================================================= -->
+          <publishMsg>${publish_msg}</publishMsg>
+          <!--============================================================= -->
         </plugin>
         <!--=============================================================== -->

File: pandora_gazebo_description/urdf/gears/sensors/thermal_sensor.gazebo.xacro (robot description, xacro)
@@ -3,5 +3,5 @@
 <!-- ###################################################################### -->
   <xacro:macro name="thermal_gazebo_sensor"
-               params="prefix_y" >
+               params="prefix_y publish_msg" >
     <gazebo reference="${prefix_y}_thermal_link" >
       <sensor name="${prefix_y}_thermal"
@@ -29,4 +29,6 @@
           <topicName>sensors/thermal</topicName> <!-- FIXME -->
           <!--============================================================= -->
+          <publishMsg>${publish_msg}</publishMsg>
+          <!--============================================================= -->
         </plugin>
         <!--=============================================================== -->
