Commit message: Add conditional when loading gazebo sensors.

File: pandora_gazebo_description/urdf/gears/gears.gazebo.xacro (robot description, xacro)
@@ -132,112 +132,136 @@
   </xacro:if>
 <!-- Load Gazebo Sensors ################################################## -->
-  <xacro:if value="${enable_gazebo_sensors}" >
-    <xacro:if value="${enable_laser_gazebo_sensor}" >
-      <xacro:laser_gazebo_sensor />
-    </xacro:if>
-    <xacro:if value="${enable_kinect_gazebo_sensor}" >
-      <xacro:kinect_gazebo_sensor />
-    </xacro:if>
-    <xacro:if value="${enable_sonar_gazebo_sensors}" >
-      <!-- ================================================================ -->
-      <xacro:if value="${enable_left_rear_sonar_gazebo_sensor}" >
-        <xacro:if value="$(arg control)" >
-          <xacro:if value="$(arg interface)" >
-            <xacro:sonar_gazebo_sensor name="left" publish_msg="false" />
-          </xacro:if>
-          <xacro:unless value="$(arg interface)" >
-            <xacro:sonar_gazebo_sensor name="left" publish_msg="true" />
+  <xacro:if value="${enable_sensors}" >
+    <xacro:if value="${enable_gazebo_sensors}" >
+      <xacro:if value="${enable_laser_sensor}" >
+        <xacro:if value="${enable_laser_gazebo_sensor}" >
+          <xacro:laser_gazebo_sensor />
+        </xacro:if>
+      </xacro:if>
+      <xacro:if value="${enable_kinect_sensor}" >
+        <xacro:if value="${enable_kinect_gazebo_sensor}" >
+          <xacro:kinect_gazebo_sensor />
+        </xacro:if>
+      </xacro:if>
+      <xacro:if value="${enable_sonar_sensors}" >
+        <xacro:if value="${enable_sonar_gazebo_sensors}" >
+          <!-- ============================================================ -->
+          <xacro:if value="${enable_left_sonar_sensor}" >
+            <xacro:if value="${enable_left_sonar_gazebo_sensor}" >
+              <xacro:if value="$(arg control)" >
+                <xacro:if value="$(arg interface)" >
+                  <xacro:sonar_gazebo_sensor name="left" publish_msg="false" />
+                </xacro:if>
+                <xacro:unless value="$(arg interface)" >
+                  <xacro:sonar_gazebo_sensor name="left" publish_msg="true" />
+                </xacro:unless>
+              </xacro:if>
+              <xacro:unless value="$(arg control)" >
+                  <xacro:sonar_gazebo_sensor name="left" publish_msg="true" />
+              </xacro:unless>
+            </xacro:if>
+          </xacro:if>
+          <!-- ============================================================ -->
+          <xacro:if value="${enable_right_sonar_sensor}" >
+            <xacro:if value="${enable_right_sonar_gazebo_sensor}" >
+              <xacro:if value="$(arg control)" >
+                <xacro:if value="$(arg interface)" >
+                  <xacro:sonar_gazebo_sensor name="right" publish_msg="false" />
+                </xacro:if>
+                <xacro:unless value="$(arg interface)" >
+                  <xacro:sonar_gazebo_sensor name="right" publish_msg="true" />
+                </xacro:unless>
+              </xacro:if>
+              <xacro:unless value="$(arg control)" >
+                  <xacro:sonar_gazebo_sensor name="right" publish_msg="true" />
+              </xacro:unless>
+            </xacro:if>
+          </xacro:if>
+          <!-- ============================================================ -->
+        </xacro:if>
+      </xacro:if>
+      <xacro:if value="${enable_co2_sensor}" >
+        <xacro:if value="${enable_co2_gazebo_sensor}" >
+          <xacro:if value="$(arg control)" >
+            <xacro:if value="$(arg interface)" >
+              <xacro:co2_gazebo_sensor publish_msg="false" />
+            </xacro:if>
+            <xacro:unless value="$(arg interface)" >
+              <xacro:co2_gazebo_sensor publish_msg="true" />
+            </xacro:unless>
+          </xacro:if>
+          <xacro:unless value="$(arg control)" >
+              <xacro:co2_gazebo_sensor publish_msg="true" />
           </xacro:unless>
         </xacro:if>
-        <xacro:unless value="$(arg control)" >
-            <xacro:sonar_gazebo_sensor name="left" publish_msg="true" />
-        </xacro:unless>
-      </xacro:if>
-      <!-- ================================================================ -->
-      <xacro:if value="${enable_right_rear_sonar_gazebo_sensor}" >
-        <xacro:if value="$(arg control)" >
-          <xacro:if value="$(arg interface)" >
-            <xacro:sonar_gazebo_sensor name="right" publish_msg="false" />
-          </xacro:if>
-          <xacro:unless value="$(arg interface)" >
-            <xacro:sonar_gazebo_sensor name="right" publish_msg="true" />
+      </xacro:if>
+      <xacro:if value="${enable_thermal_sensors}" >
+        <xacro:if value="${enable_thermal_gazebo_sensors}" >
+          <!-- ============================================================ -->
+          <xacro:if value="${enable_middle_thermal_sensor}" >
+            <xacro:if value="${enable_middle_thermal_gazebo_sensor}" >
+              <xacro:if value="$(arg control)" >
+                <xacro:if value="$(arg interface)" >
+                  <xacro:thermal_gazebo_sensor prefix_y="middle" publish_msg="false" />
+                </xacro:if>
+                <xacro:unless value="$(arg interface)" >
+                  <xacro:thermal_gazebo_sensor prefix_y="middle" publish_msg="true" />
+                </xacro:unless>
+              </xacro:if>
+              <xacro:unless value="$(arg control)" >
+                  <xacro:thermal_gazebo_sensor prefix_y="middle" publish_msg="true" />
+              </xacro:unless>
+            </xacro:if>
+          </xacro:if>
+          <!-- ============================================================ -->
+          <xacro:if value="${enable_left_thermal_sensor}" >
+            <xacro:if value="${enable_left_thermal_gazebo_sensor}" >
+              <xacro:if value="$(arg control)" >
+                <xacro:if value="$(arg interface)" >
+                  <xacro:thermal_gazebo_sensor prefix_y="left" publish_msg="false" />
+                </xacro:if>
+                <xacro:unless value="$(arg interface)" >
+                  <xacro:thermal_gazebo_sensor prefix_y="left" publish_msg="true" />
+                </xacro:unless>
+              </xacro:if>
+              <xacro:unless value="$(arg control)" >
+                  <xacro:thermal_gazebo_sensor prefix_y="left" publish_msg="true" />
+              </xacro:unless>
+            </xacro:if>
+          </xacro:if>
+          <!-- ============================================================ -->
+          <xacro:if value="${enable_right_thermal_sensor}" >
+            <xacro:if value="${enable_right_thermal_gazebo_sensor}" >
+              <xacro:if value="$(arg control)" >
+                <xacro:if value="$(arg interface)" >
+                  <xacro:thermal_gazebo_sensor prefix_y="right" publish_msg="false" />
+                </xacro:if>
+                <xacro:unless value="$(arg interface)" >
+                  <xacro:thermal_gazebo_sensor prefix_y="right" publish_msg="true" />
+                </xacro:unless>
+              </xacro:if>
+              <xacro:unless value="$(arg control)" >
+                  <xacro:thermal_gazebo_sensor prefix_y="right" publish_msg="true" />
+              </xacro:unless>
+            </xacro:if>
+          </xacro:if>
+          <!-- ============================================================ -->
+        </xacro:if>
+      </xacro:if>
+      <xacro:if value="${enable_microphone_sensor}" >
+        <xacro:if value="${enable_microphone_gazebo_sensor}" >
+          <xacro:if value="$(arg control)" >
+            <xacro:if value="$(arg interface)" >
+              <xacro:microphone_gazebo_sensor publish_msg="false" />
+            </xacro:if>
+            <xacro:unless value="$(arg interface)" >
+              <xacro:microphone_gazebo_sensor publish_msg="true" />
+            </xacro:unless>
+          </xacro:if>
+          <xacro:unless value="$(arg control)" >
+              <xacro:microphone_gazebo_sensor publish_msg="true" />
           </xacro:unless>
         </xacro:if>
-        <xacro:unless value="$(arg control)" >
-            <xacro:sonar_gazebo_sensor name="right" publish_msg="true" />
-        </xacro:unless>
-      </xacro:if>
-      <!-- ================================================================ -->
-    </xacro:if>
-    <xacro:if value="${enable_co2_gazebo_sensor}" >
-      <xacro:if value="$(arg control)" >
-        <xacro:if value="$(arg interface)" >
-          <xacro:co2_gazebo_sensor publish_msg="false" />
-        </xacro:if>
-        <xacro:unless value="$(arg interface)" >
-          <xacro:co2_gazebo_sensor publish_msg="true" />
-        </xacro:unless>
-      </xacro:if>
-      <xacro:unless value="$(arg control)" >
-          <xacro:co2_gazebo_sensor publish_msg="true" />
-      </xacro:unless>
-    </xacro:if>
-    <xacro:if value="${enable_thermal_gazebo_sensors}" >
-      <!-- ================================================================ -->
-      <xacro:if value="${enable_middle_thermal_gazebo_sensor}" >
-        <xacro:if value="$(arg control)" >
-          <xacro:if value="$(arg interface)" >
-            <xacro:thermal_gazebo_sensor prefix_y="middle" publish_msg="false" />
-          </xacro:if>
-          <xacro:unless value="$(arg interface)" >
-            <xacro:thermal_gazebo_sensor prefix_y="middle" publish_msg="true" />
-          </xacro:unless>
-        </xacro:if>
-        <xacro:unless value="$(arg control)" >
-            <xacro:thermal_gazebo_sensor prefix_y="middle" publish_msg="true" />
-        </xacro:unless>
-      </xacro:if>
-      <!-- ================================================================ -->
-      <xacro:if value="${enable_left_thermal_gazebo_sensor}" >
-        <xacro:if value="$(arg control)" >
-          <xacro:if value="$(arg interface)" >
-            <xacro:thermal_gazebo_sensor prefix_y="left" publish_msg="false" />
-          </xacro:if>
-          <xacro:unless value="$(arg interface)" >
-            <xacro:thermal_gazebo_sensor prefix_y="left" publish_msg="true" />
-          </xacro:unless>
-        </xacro:if>
-        <xacro:unless value="$(arg control)" >
-            <xacro:thermal_gazebo_sensor prefix_y="left" publish_msg="true" />
-        </xacro:unless>
-      </xacro:if>
-      <!-- ================================================================ -->
-      <xacro:if value="${enable_right_thermal_gazebo_sensor}" >
-        <xacro:if value="$(arg control)" >
-          <xacro:if value="$(arg interface)" >
-            <xacro:thermal_gazebo_sensor prefix_y="right" publish_msg="false" />
-          </xacro:if>
-          <xacro:unless value="$(arg interface)" >
-            <xacro:thermal_gazebo_sensor prefix_y="right" publish_msg="true" />
-          </xacro:unless>
-        </xacro:if>
-        <xacro:unless value="$(arg control)" >
-            <xacro:thermal_gazebo_sensor prefix_y="right" publish_msg="true" />
-        </xacro:unless>
-      </xacro:if>
-      <!-- ================================================================ -->
-    </xacro:if>
-    <xacro:if value="${enable_microphone_gazebo_sensor}" >
-      <xacro:if value="$(arg control)" >
-        <xacro:if value="$(arg interface)" >
-          <xacro:microphone_gazebo_sensor publish_msg="false" />
-        </xacro:if>
-        <xacro:unless value="$(arg interface)" >
-          <xacro:microphone_gazebo_sensor publish_msg="true" />
-        </xacro:unless>
-      </xacro:if>
-      <xacro:unless value="$(arg control)" >
-          <xacro:microphone_gazebo_sensor publish_msg="true" />
-      </xacro:unless>
+      </xacro:if>
     </xacro:if>
   </xacro:if>

File: pandora_gazebo_description/urdf/gears/sdf_configurations.xacro (robot description, xacro)
@@ -17,6 +17,6 @@
     <!-- ================================================================== -->
     <xacro:property name="enable_sonar_gazebo_sensors" value="true" />
-      <xacro:property name="enable_left_rear_sonar_gazebo_sensor" value="true" />
-      <xacro:property name="enable_right_rear_sonar_gazebo_sensor" value="true" />
+      <xacro:property name="enable_left_sonar_gazebo_sensor" value="true" />
+      <xacro:property name="enable_right_sonar_gazebo_sensor" value="true" />
     <!-- ================================================================== -->
     <xacro:property name="enable_thermal_gazebo_sensors" value="true" />

Commit message: Adjust wheel physics (first attempt).

File: pandora_gazebo_description/urdf/gears/gears.gazebo.xacro (robot description, xacro)
@@ -390,17 +390,15 @@
       </xacro:if>
     </xacro:unless>
-    <xacro:if value="$(arg control)" >
-      <!-- ================================================================ -->
-      <xacro:if value="$(arg interface)" >
-        <xacro:gazebo_ros_control_plugin namespace="/"
-                                         hardware_interface="pandora_gazebo_interface/GazeboInterface" />
-      </xacro:if>
-      <!-- ================================================================ -->
-      <xacro:unless value="$(arg interface)" >
-        <xacro:gazebo_ros_control_plugin namespace="/"
-                                         hardware_interface="gazebo_ros_control/DefaultRobotHWSim" />
-      </xacro:unless>
-      <!-- ================================================================ -->
-    </xacro:if>
+  </xacro:if>
+<!-- Load Ros Control ##################################################### -->
+  <xacro:if value="$(arg control)" >
+    <xacro:if value="$(arg interface)" >
+      <xacro:gazebo_ros_control_plugin namespace="/"
+                                       hardware_interface="pandora_gazebo_interface/GazeboInterface" />
+    </xacro:if>
+    <xacro:unless value="$(arg interface)" >
+      <xacro:gazebo_ros_control_plugin namespace="/"
+                                       hardware_interface="gazebo_ros_control/DefaultRobotHWSim" />
+    </xacro:unless>
   </xacro:if>
 <!-- ###################################################################### -->

File: pandora_gazebo_description/urdf/gears/gears_simplified.gazebo.xacro (robot description, xacro)
@@ -21,10 +21,12 @@
   <xacro:include filename="$(find pandora_gazebo_description)/urdf/gears/plugins/ros_control_plugin.gazebo.xacro" />
 <!-- Properties ########################################################### -->
+  <!-- XXX: Get from config -->
   <xacro:property name="robot_namespace" value="" />
-  <xacro:property name="wheel_mu_1" value="0.75" />
-  <xacro:property name="wheel_mu_2" value="0.75" />
+  <xacro:property name="wheel_mu_1" value="0.675" />
+  <xacro:property name="wheel_mu_2" value="0.675" />
   <xacro:property name="wheel_k_p" value="10000000.0" />
-  <xacro:property name="wheel_k_d" value="1.0" />
+  <xacro:property name="wheel_k_d" value="0.8" />
   <xacro:property name="wheel_min_depth" value="0.001" />
+  <xacro:property name="wheel_max_contacts" value="1" />
 <!-- Load URDF ############################################################ -->
   <xacro:gears_urdf fixed="false" />

File: pandora_gazebo_description/urdf/gears/physics/wheel_link_physics.gazebo.xacro (robot description, xacro)
@@ -26,5 +26,5 @@
       <!-- <selfCollide>false</selfCollide> -->
       <!-- ================================================================ -->
-      <maxContacts>1</maxContacts>
+      <maxContacts>${wheel_max_contacts}</maxContacts>
       <!-- ================================================================ -->
       <!-- <laserRetro>0</laserRetro> -->

File: pandora_gazebo_description/urdf/gears/sdf_configurations.xacro (robot description, xacro)
@@ -65,9 +65,10 @@
 <!-- Joint Physics ######################################################## -->
   <!-- Wheels ============================================================= -->
-  <xacro:property name="wheel_mu_1" value="0.75" />
-  <xacro:property name="wheel_mu_2" value="0.75" />
+  <xacro:property name="wheel_mu_1" value="0.675" />
+  <xacro:property name="wheel_mu_2" value="0.675" />
   <xacro:property name="wheel_k_p" value="10000000.0" />
-  <xacro:property name="wheel_k_d" value="1.0" />
+  <xacro:property name="wheel_k_d" value="0.8" />
   <xacro:property name="wheel_min_depth" value="0.001" />
+  <xacro:property name="wheel_max_contacts" value="1" />
   <!-- ==================================================================== -->
 <!-- Plugin Parameters #################################################### -->
