Commit message: Finalize camera sensors.

File: pandora_gazebo_description/urdf/gears/gears.gazebo.xacro (robot description, xacro)
@@ -24,4 +24,5 @@
   <xacro:include filename="$(find pandora_gazebo_description)/urdf/gears/sensors/laser_sensor.gazebo.xacro" />
   <xacro:include filename="$(find pandora_gazebo_description)/urdf/gears/sensors/kinect_sensor.gazebo.xacro" />
+  <xacro:include filename="$(find pandora_gazebo_description)/urdf/gears/sensors/camera_sensor.gazebo.xacro" />
   <xacro:include filename="$(find pandora_gazebo_description)/urdf/gears/sensors/sonar_sensor.gazebo.xacro" />
   <xacro:include filename="$(find pandora_gazebo_description)/urdf/gears/sensors/thermal_sensor.gazebo.xacro" />
@@ -128,4 +129,21 @@
         </xacro:if>
       </xacro:if>
+      <xacro:if value="${enable_camera_sensors}" >
+        <xacro:if value="${enable_camera_gazebo_sensors}" >
+          <!-- ============================================================ -->
+          <xacro:if value="${enable_left_camera_sensor}" >
+            <xacro:if value="${enable_left_camera_gazebo_sensor}" >
+              <xacro:camera_gazebo_sensor prefix_y="left" />
+            </xacro:if>
+          </xacro:if>
+          <!-- ============================================================ -->
+          <xacro:if value="${enable_right_camera_sensor}" >
+            <xacro:if value="${enable_right_camera_gazebo_sensor}" >
+              <xacro:camera_gazebo_sensor prefix_y="right" />
+            </xacro:if>
+          </xacro:if>
+          <!-- ============================================================ -->
+        </xacro:if>
+      </xacro:if>
       <xacro:if value="${enable_sonar_sensors}" >
         <xacro:if value="${enable_sonar_gazebo_sensors}" >
@@ -135,12 +153,12 @@
               <xacro:if value="$(arg control)" >
                 <xacro:if value="$(arg interface)" >
-                    <xacro:sonar_gazebo_sensor name="left" publish_msg="false" />
+                  <xacro:sonar_gazebo_sensor prefix_y="left" publish_msg="false" />
                 </xacro:if>
                 <xacro:unless value="$(arg interface)" >
-                    <xacro:sonar_gazebo_sensor name="left" publish_msg="true" />
+                  <xacro:sonar_gazebo_sensor prefix_y="left" publish_msg="true" />
                 </xacro:unless>
               </xacro:if>
               <xacro:unless value="$(arg control)" >
-                  <xacro:sonar_gazebo_sensor name="left" publish_msg="true" />
+                <xacro:sonar_gazebo_sensor prefix_y="left" publish_msg="true" />
               </xacro:unless>
             </xacro:if>
@@ -151,12 +169,12 @@
               <xacro:if value="$(arg control)" >
                 <xacro:if value="$(arg interface)" >
-                    <xacro:sonar_gazebo_sensor name="right" publish_msg="false" />
+                  <xacro:sonar_gazebo_sensor prefix_y="right" publish_msg="false" />
                 </xacro:if>
                 <xacro:unless value="$(arg interface)" >
-                    <xacro:sonar_gazebo_sensor name="right" publish_msg="true" />
+                  <xacro:sonar_gazebo_sensor prefix_y="right" publish_msg="true" />
                 </xacro:unless>
               </xacro:if>
               <xacro:unless value="$(arg control)" >
-                  <xacro:sonar_gazebo_sensor name="right" publish_msg="true" />
+                <xacro:sonar_gazebo_sensor prefix_y="right" publish_msg="true" />
               </xacro:unless>
             </xacro:if>

File: pandora_gazebo_description/urdf/gears/gears_simplified.gazebo.xacro (robot description, xacro)
@@ -8,4 +8,5 @@
   <xacro:include filename="$(find pandora_gazebo_description)/urdf/gears/sensors/laser_sensor.gazebo.xacro" />
   <xacro:include filename="$(find pandora_gazebo_description)/urdf/gears/sensors/kinect_sensor.gazebo.xacro" />
+  <xacro:include filename="$(find pandora_gazebo_description)/urdf/gears/sensors/camera_sensor.gazebo.xacro" />
   <xacro:include filename="$(find pandora_gazebo_description)/urdf/gears/sensors/sonar_sensor.gazebo.xacro" />
   <xacro:include filename="$(find pandora_gazebo_description)/urdf/gears/sensors/thermal_sensor.gazebo.xacro" />
@@ -40,6 +41,8 @@
   <xacro:laser_gazebo_sensor />
   <xacro:kinect_gazebo_sensor />
-  <xacro:sonar_gazebo_sensor name="left" publish_msg="false" />
-  <xacro:sonar_gazebo_sensor name="right" publish_msg="false" />
+  <xacro:camera_gazebo_sensor prefix_y="left" />
+  <xacro:camera_gazebo_sensor prefix_y="right" />
+  <xacro:sonar_gazebo_sensor prefix_y="left" publish_msg="false" />
+  <xacro:sonar_gazebo_sensor prefix_y="right" publish_msg="false" />
   <xacro:co2_gazebo_sensor publish_msg="false" publish_viz="false" />
   <xacro:thermal_gazebo_sensor prefix_y="middle" publish_msg="false" publish_viz="false" />

File: pandora_gazebo_description/urdf/gears/sdf_configurations.xacro (robot description, xacro)
@@ -15,4 +15,8 @@
     <!-- ================================================================== -->
     <xacro:property name="enable_kinect_gazebo_sensor" value="true" />
+    <!-- ================================================================== -->
+    <xacro:property name="enable_camera_gazebo_sensors" value="true" />
+      <xacro:property name="enable_left_camera_gazebo_sensor" value="true" />
+      <xacro:property name="enable_right_camera_gazebo_sensor" value="true" />
     <!-- ================================================================== -->
     <xacro:property name="enable_sonar_gazebo_sensors" value="true" />
@@ -65,9 +69,9 @@
 <!-- Joint Physics ######################################################## -->
   <!-- Wheels ============================================================= -->
-  <xacro:property name="wheel_mu_1" value="0.65" />
-  <xacro:property name="wheel_mu_2" value="0.65" />
-  <xacro:property name="wheel_k_p" value="100000000.0" />
-  <xacro:property name="wheel_k_d" value="0.8" />
-  <xacro:property name="wheel_min_depth" value="0.00001" />
+  <xacro:property name="wheel_mu_1" value="0.45" />
+  <xacro:property name="wheel_mu_2" value="0.45" />
+  <xacro:property name="wheel_k_p" value="10000000.0" />
+  <xacro:property name="wheel_k_d" value="1.0" />
+  <xacro:property name="wheel_min_depth" value="0.0001" />
   <xacro:property name="wheel_max_contacts" value="1" />
   <!-- ==================================================================== -->

File: pandora_gazebo_description/urdf/gears/sensors/camera_sensor.gazebo.xacro (robot description, xacro)
@@ -2,7 +2,7 @@
 <robot xmlns:xacro="http://ros.org/wiki/xacro" >
 <!-- ###################################################################### -->
-  <xacro:macro name="logitech_gazebo_sensor"
+  <xacro:macro name="camera_gazebo_sensor"
                params="prefix_y" >
-    <gazebo reference="${prefix_y}_camera_link" >
+    <gazebo reference="${prefix_y}_camera_frame" >
       <sensor name="${prefix_y}_camera"
               type="camera" >
@@ -14,4 +14,5 @@
             <width>1280</width>
             <height>720</height>
+            <format>R8G8B8</format> <!-- FIXME -->
           </image>
           <!--============================================================= -->
@@ -25,7 +26,7 @@
                 filename="libgazebo_ros_camera.so" >
           <!--============================================================= -->
-          <frameName>${prefix_y}_camera_link</frameName>
+          <frameName>${prefix_y}_camera_optical_frame</frameName>
           <!--============================================================= -->
-          <topicName>${prefix_y}_camera/image</topicName>
+          <imageTopicName>${prefix_y}_camera/image</imageTopicName>
           <!--============================================================= -->
         </plugin>
@@ -33,5 +34,5 @@
         <always_on>1</always_on>
         <!--=============================================================== -->
-        <update_rate>5</update_rate>
+        <update_rate>5</update_rate> <!-- FIXME -->
         <!--=============================================================== -->
         <visualize>false</visualize>

File: pandora_gazebo_description/urdf/gears/sensors/sonar_sensor.gazebo.xacro (robot description, xacro)
@@ -3,7 +3,7 @@
 <!-- ###################################################################### -->
   <xacro:macro name="sonar_gazebo_sensor"
-               params="name publish_msg" >
-    <gazebo reference="${name}_sonar_link" >
-      <sensor name="${name}_sonar"
+               params="prefix_y publish_msg" >
+    <gazebo reference="${prefix_y}_sonar_link" >
+      <sensor name="${prefix_y}_sonar"
               type="ray" >
         <!--=============================================================== -->
@@ -42,5 +42,5 @@
           <robotNamespace></robotNamespace>
           <!--============================================================= -->
-          <frameName>${name}_sonar_link</frameName>
+          <frameName>${prefix_y}_sonar_link</frameName>
           <!--============================================================= -->
           <topicName>/sensors/sonar</topicName> <!-- FIXME -->

Commit message: Add linear sonar sensor in urdf & xmega interface.

File: pandora_gazebo_description/urdf/gears/gears.gazebo.xacro (robot description, xacro)
@@ -149,16 +149,32 @@
         <xacro:if value="${enable_sonar_gazebo_sensors}" >
           <!-- ============================================================ -->
+          <xacro:if value="${enable_linear_sonar_sensor}" >
+            <xacro:if value="${enable_linear_sonar_gazebo_sensor}" >
+              <xacro:if value="$(arg control)" >
+                <xacro:if value="$(arg interface)" >
+                  <xacro:sonar_gazebo_sensor name="linear" publish_msg="false" />
+                </xacro:if>
+                <xacro:unless value="$(arg interface)" >
+                  <xacro:sonar_gazebo_sensor name="linear" publish_msg="true" />
+                </xacro:unless>
+              </xacro:if>
+              <xacro:unless value="$(arg control)" >
+                <xacro:sonar_gazebo_sensor name="linear" publish_msg="true" />
+              </xacro:unless>
+            </xacro:if>
+          </xacro:if>
+          <!-- ============================================================ -->
           <xacro:if value="${enable_left_sonar_sensor}" >
             <xacro:if value="${enable_left_sonar_gazebo_sensor}" >
               <xacro:if value="$(arg control)" >
                 <xacro:if value="$(arg interface)" >
-                  <xacro:sonar_gazebo_sensor prefix_y="left" publish_msg="false" />
-                </xacro:if>
-                <xacro:unless value="$(arg interface)" >
-                  <xacro:sonar_gazebo_sensor prefix_y="left" publish_msg="true" />
-                </xacro:unless>
-              </xacro:if>
-              <xacro:unless value="$(arg control)" >
-                <xacro:sonar_gazebo_sensor prefix_y="left" publish_msg="true" />
+                  <xacro:sonar_gazebo_sensor name="left" publish_msg="false" />
+                </xacro:if>
+                <xacro:unless value="$(arg interface)" >
+                  <xacro:sonar_gazebo_sensor name="left" publish_msg="true" />
+                </xacro:unless>
+              </xacro:if>
+              <xacro:unless value="$(arg control)" >
+                <xacro:sonar_gazebo_sensor name="left" publish_msg="true" />
               </xacro:unless>
             </xacro:if>
@@ -169,12 +185,12 @@
               <xacro:if value="$(arg control)" >
                 <xacro:if value="$(arg interface)" >
-                  <xacro:sonar_gazebo_sensor prefix_y="right" publish_msg="false" />
-                </xacro:if>
-                <xacro:unless value="$(arg interface)" >
-                  <xacro:sonar_gazebo_sensor prefix_y="right" publish_msg="true" />
-                </xacro:unless>
-              </xacro:if>
-              <xacro:unless value="$(arg control)" >
-                <xacro:sonar_gazebo_sensor prefix_y="right" publish_msg="true" />
+                  <xacro:sonar_gazebo_sensor name="right" publish_msg="false" />
+                </xacro:if>
+                <xacro:unless value="$(arg interface)" >
+                  <xacro:sonar_gazebo_sensor name="right" publish_msg="true" />
+                </xacro:unless>
+              </xacro:if>
+              <xacro:unless value="$(arg control)" >
+                <xacro:sonar_gazebo_sensor name="right" publish_msg="true" />
               </xacro:unless>
             </xacro:if>

File: pandora_gazebo_description/urdf/gears/gears_simplified.gazebo.xacro (robot description, xacro)
@@ -43,6 +43,7 @@
   <xacro:camera_gazebo_sensor prefix_y="left" />
   <xacro:camera_gazebo_sensor prefix_y="right" />
-  <xacro:sonar_gazebo_sensor prefix_y="left" publish_msg="false" />
-  <xacro:sonar_gazebo_sensor prefix_y="right" publish_msg="false" />
+  <xacro:sonar_gazebo_sensor name="linear" publish_msg="false" />
+  <xacro:sonar_gazebo_sensor name="left" publish_msg="false" />
+  <xacro:sonar_gazebo_sensor name="right" publish_msg="false" />
   <xacro:co2_gazebo_sensor publish_msg="false" publish_viz="false" />
   <xacro:thermal_gazebo_sensor prefix_y="middle" publish_msg="false" publish_viz="false" />

File: pandora_gazebo_description/urdf/gears/sdf_configurations.xacro (robot description, xacro)
@@ -21,4 +21,5 @@
     <!-- ================================================================== -->
     <xacro:property name="enable_sonar_gazebo_sensors" value="true" />
+      <xacro:property name="enable_linear_sonar_gazebo_sensor" value="true" />
       <xacro:property name="enable_left_sonar_gazebo_sensor" value="true" />
       <xacro:property name="enable_right_sonar_gazebo_sensor" value="true" />
@@ -69,9 +70,9 @@
 <!-- Joint Physics ######################################################## -->
   <!-- Wheels ============================================================= -->
-  <xacro:property name="wheel_mu_1" value="0.675" />
-  <xacro:property name="wheel_mu_2" value="0.675" />
-  <xacro:property name="wheel_k_p" value="100000000.0" />
-  <xacro:property name="wheel_k_d" value="0.8" />
-  <xacro:property name="wheel_min_depth" value="0.00001" />
+  <xacro:property name="wheel_mu_1" value="0.6" />
+  <xacro:property name="wheel_mu_2" value="0.3" />
+  <xacro:property name="wheel_k_p" value="10000000.0" />
+  <xacro:property name="wheel_k_d" value="1.0" />
+  <xacro:property name="wheel_min_depth" value="0.0001" />
   <xacro:property name="wheel_max_contacts" value="1" />
   <!-- ==================================================================== -->

File: pandora_gazebo_description/urdf/gears/sensors/sonar_sensor.gazebo.xacro (robot description, xacro)
@@ -3,7 +3,7 @@
 <!-- ###################################################################### -->
   <xacro:macro name="sonar_gazebo_sensor"
-               params="prefix_y publish_msg" >
-    <gazebo reference="${prefix_y}_sonar_frame" >
-      <sensor name="${prefix_y}_sonar"
+               params="name publish_msg" >
+    <gazebo reference="${name}_sonar_frame" >
+      <sensor name="${name}_sonar"
               type="ray" >
         <ray>
@@ -39,5 +39,5 @@
           <robotNamespace></robotNamespace>
           <!--============================================================= -->
-          <frameName>${prefix_y}_sonar_frame</frameName>
+          <frameName>${name}_sonar_frame</frameName>
           <!--============================================================= -->
           <topicName>/sensors/sonar</topicName> <!-- FIXME -->
