Commit message: Remove args to publish msg and viz from sensor plugins

File: pandora_gazebo_description/urdf/gears/gears.gazebo.xacro (robot description, xacro)
@@ -153,15 +153,5 @@
           <xacro:if value="${enable_linear_sonar_sensor}" >
             <xacro:if value="${enable_linear_sonar_gazebo_sensor}" >
-              <xacro:if value="$(arg control)" >
-                <xacro:if value="$(arg interface)" >
-                  <xacro:sonar_gazebo_sensor name="linear" publish_msg="false" />
-                </xacro:if>
-                <xacro:unless value="$(arg interface)" >
-                  <xacro:sonar_gazebo_sensor name="linear" publish_msg="true" />
-                </xacro:unless>
-              </xacro:if>
-              <xacro:unless value="$(arg control)" >
-                <xacro:sonar_gazebo_sensor name="linear" publish_msg="true" />
-              </xacro:unless>
+              <xacro:sonar_gazebo_sensor name="linear" />
             </xacro:if>
           </xacro:if>
@@ -169,15 +159,5 @@
           <xacro:if value="${enable_left_sonar_sensor}" >
             <xacro:if value="${enable_left_sonar_gazebo_sensor}" >
-              <xacro:if value="$(arg control)" >
-                <xacro:if value="$(arg interface)" >
-                  <xacro:sonar_gazebo_sensor name="left" publish_msg="false" />
-                </xacro:if>
-                <xacro:unless value="$(arg interface)" >
-                  <xacro:sonar_gazebo_sensor name="left" publish_msg="true" />
-                </xacro:unless>
-              </xacro:if>
-              <xacro:unless value="$(arg control)" >
-                <xacro:sonar_gazebo_sensor name="left" publish_msg="true" />
-              </xacro:unless>
+                  <xacro:sonar_gazebo_sensor name="left" />
             </xacro:if>
           </xacro:if>
@@ -185,15 +165,5 @@
           <xacro:if value="${enable_right_sonar_sensor}" >
             <xacro:if value="${enable_right_sonar_gazebo_sensor}" >
-              <xacro:if value="$(arg control)" >
-                <xacro:if value="$(arg interface)" >
-                  <xacro:sonar_gazebo_sensor name="right" publish_msg="false" />
-                </xacro:if>
-                <xacro:unless value="$(arg interface)" >
-                  <xacro:sonar_gazebo_sensor name="right" publish_msg="true" />
-                </xacro:unless>
-              </xacro:if>
-              <xacro:unless value="$(arg control)" >
-                <xacro:sonar_gazebo_sensor name="right" publish_msg="true" />
-              </xacro:unless>
+                  <xacro:sonar_gazebo_sensor name="right" />
             </xacro:if>
           </xacro:if>
@@ -203,30 +173,5 @@
       <xacro:if value="${enable_co2_sensor}" >
         <xacro:if value="${enable_co2_gazebo_sensor}" >
-          <xacro:if value="$(arg control)" >
-            <xacro:if value="$(arg interface)" >
-              <xacro:if value="$(arg sensors_viz)" >
-                <xacro:co2_gazebo_sensor publish_msg="false" publish_viz="true" />
-              </xacro:if>
-              <xacro:unless value="$(arg sensors_viz)" >
-                <xacro:co2_gazebo_sensor publish_msg="false" publish_viz="false" />
-              </xacro:unless>
-            </xacro:if>
-            <xacro:unless value="$(arg interface)" >
-              <xacro:if value="$(arg sensors_viz)" >
-                <xacro:co2_gazebo_sensor publish_msg="true" publish_viz="true" />
-              </xacro:if>
-              <xacro:unless value="$(arg sensors_viz)" >
-                <xacro:co2_gazebo_sensor publish_msg="true" publish_viz="false" />
-              </xacro:unless>
-            </xacro:unless>
-          </xacro:if>
-          <xacro:unless value="$(arg control)" >
-            <xacro:if value="$(arg sensors_viz)" >
-              <xacro:co2_gazebo_sensor publish_msg="true" publish_viz="true" />
-            </xacro:if>
-            <xacro:unless value="$(arg sensors_viz)" >
-              <xacro:co2_gazebo_sensor publish_msg="true" publish_viz="false" />
-            </xacro:unless>
-          </xacro:unless>
+                <xacro:co2_gazebo_sensor />
         </xacro:if>
       </xacro:if>
@@ -236,30 +181,5 @@
           <xacro:if value="${enable_middle_thermal_sensor}" >
             <xacro:if value="${enable_middle_thermal_gazebo_sensor}" >
-              <xacro:if value="$(arg control)" >
-                <xacro:if value="$(arg interface)" >
-                  <xacro:if value="$(arg sensors_viz)" >
-                    <xacro:thermal_gazebo_sensor prefix_y="middle" publish_msg="false" publish_viz="true" />
-                  </xacro:if>
-                  <xacro:unless value="$(arg sensors_viz)" >
-                    <xacro:thermal_gazebo_sensor prefix_y="middle" publish_msg="false" publish_viz="false" />
-                  </xacro:unless>
-                </xacro:if>
-                <xacro:unless value="$(arg interface)" >
-                  <xacro:if value="$(arg sensors_viz)" >
-                    <xacro:thermal_gazebo_sensor prefix_y="middle" publish_msg="true" publish_viz="true" />
-                  </xacro:if>
-                  <xacro:unless value="$(arg sensors_viz)" >
-                    <xacro:thermal_gazebo_sensor prefix_y="middle" publish_msg="true" publish_viz="false" />
-                  </xacro:unless>
-                </xacro:unless>
-              </xacro:if>
-              <xacro:unless value="$(arg control)" >
-                <xacro:if value="$(arg sensors_viz)" >
-                  <xacro:thermal_gazebo_sensor prefix_y="middle" publish_msg="true" publish_viz="true" />
-                </xacro:if>
-                <xacro:unless value="$(arg sensors_viz)" >
-                  <xacro:thermal_gazebo_sensor prefix_y="middle" publish_msg="true" publish_viz="false" />
-                </xacro:unless>
-              </xacro:unless>
+                    <xacro:thermal_gazebo_sensor prefix_y="middle" />
             </xacro:if>
           </xacro:if>
@@ -267,30 +187,5 @@
           <xacro:if value="${enable_left_thermal_sensor}" >
             <xacro:if value="${enable_left_thermal_gazebo_sensor}" >
-              <xacro:if value="$(arg control)" >
-                <xacro:if value="$(arg interface)" >
-                  <xacro:if value="$(arg sensors_viz)" >
-                    <xacro:thermal_gazebo_sensor prefix_y="left" publish_msg="false" publish_viz="true" />
-                  </xacro:if>
-                  <xacro:unless value="$(arg sensors_viz)" >
-                    <xacro:thermal_gazebo_sensor prefix_y="left" publish_msg="false" publish_viz="false" />
-                  </xacro:unless>
-                </xacro:if>
-                <xacro:unless value="$(arg interface)" >
-                  <xacro:if value="$(arg sensors_viz)" >
-                    <xacro:thermal_gazebo_sensor prefix_y="left" publish_msg="true" publish_viz="true" />
-                  </xacro:if>
-                  <xacro:unless value="$(arg sensors_viz)" >
-                    <xacro:thermal_gazebo_sensor prefix_y="left" publish_msg="true" publish_viz="false" />
-                  </xacro:unless>
-                </xacro:unless>
-              </xacro:if>
-              <xacro:unless value="$(arg control)" >
-                <xacro:if value="$(arg sensors_viz)" >
-                  <xacro:thermal_gazebo_sensor prefix_y="left" publish_msg="true" publish_viz="true" />
-                </xacro:if>
-                <xacro:unless value="$(arg sensors_viz)" >
-                  <xacro:thermal_gazebo_sensor prefix_y="left" publish_msg="true" publish_viz="false" />
-                </xacro:unless>
-              </xacro:unless>
+                    <xacro:thermal_gazebo_sensor prefix_y="left" />
             </xacro:if>
           </xacro:if>
@@ -298,30 +193,5 @@
           <xacro:if value="${enable_right_thermal_sensor}" >
             <xacro:if value="${enable_right_thermal_gazebo_sensor}" >
-              <xacro:if value="$(arg control)" >
-                <xacro:if value="$(arg interface)" >
-                  <xacro:if value="$(arg sensors_viz)" >
-                    <xacro:thermal_gazebo_sensor prefix_y="right" publish_msg="false" publish_viz="true" />
-                  </xacro:if>
-                  <xacro:unless value="$(arg sensors_viz)" >
-                    <xacro:thermal_gazebo_sensor prefix_y="right" publish_msg="false" publish_viz="false" />
-                  </xacro:unless>
-                </xacro:if>
-                <xacro:unless value="$(arg interface)" >
-                  <xacro:if value="$(arg sensors_viz)" >
-                    <xacro:thermal_gazebo_sensor prefix_y="right" publish_msg="true" publish_viz="true" />
-                  </xacro:if>
-                  <xacro:unless value="$(arg sensors_viz)" >
-                    <xacro:thermal_gazebo_sensor prefix_y="right" publish_msg="true" publish_viz="false" />
-                  </xacro:unless>
-                </xacro:unless>
-              </xacro:if>
-              <xacro:unless value="$(arg control)" >
-                <xacro:if value="$(arg sensors_viz)" >
-                  <xacro:thermal_gazebo_sensor prefix_y="right" publish_msg="true" publish_viz="true" />
-                </xacro:if>
-                <xacro:unless value="$(arg sensors_viz)" >
-                  <xacro:thermal_gazebo_sensor prefix_y="right" publish_msg="true" publish_viz="false" />
-                </xacro:unless>
-              </xacro:unless>
+                    <xacro:thermal_gazebo_sensor prefix_y="right" />
             </xacro:if>
           </xacro:if>
@@ -331,30 +201,5 @@
       <xacro:if value="${enable_microphone_sensor}" >
         <xacro:if value="${enable_microphone_gazebo_sensor}" >
-          <xacro:if value="$(arg control)" >
-            <xacro:if value="$(arg interface)" >
-              <xacro:if value="$(arg sensors_viz)" >
-                <xacro:microphone_gazebo_sensor publish_msg="false" publish_viz="true" />
-              </xacro:if>
-              <xacro:unless value="$(arg sensors_viz)" >
-                <xacro:microphone_gazebo_sensor publish_msg="false" publish_viz="false" />
-              </xacro:unless>
-            </xacro:if>
-            <xacro:unless value="$(arg interface)" >
-              <xacro:if value="$(arg sensors_viz)" >
-                <xacro:microphone_gazebo_sensor publish_msg="true" publish_viz="true" />
-              </xacro:if>
-              <xacro:unless value="$(arg sensors_viz)" >
-                <xacro:microphone_gazebo_sensor publish_msg="true" publish_viz="false" />
-              </xacro:unless>
-            </xacro:unless>
-          </xacro:if>
-          <xacro:unless value="$(arg control)" >
-            <xacro:if value="$(arg sensors_viz)" >
-              <xacro:microphone_gazebo_sensor publish_msg="true" publish_viz="true" />
-            </xacro:if>
-            <xacro:unless value="$(arg sensors_viz)" >
-              <xacro:microphone_gazebo_sensor publish_msg="true" publish_viz="false" />
-            </xacro:unless>
-          </xacro:unless>
+                <xacro:microphone_gazebo_sensor />
         </xacro:if>
       </xacro:if>

File: pandora_gazebo_description/urdf/gears/gears_simplified.gazebo.xacro (robot description, xacro)
@@ -45,12 +45,12 @@
   <xacro:camera_gazebo_sensor prefix_y="left" />
   <xacro:camera_gazebo_sensor prefix_y="right" />
-  <xacro:sonar_gazebo_sensor name="linear" publish_msg="false" />
-  <xacro:sonar_gazebo_sensor name="left" publish_msg="false" />
-  <xacro:sonar_gazebo_sensor name="right" publish_msg="false" />
-  <xacro:co2_gazebo_sensor publish_msg="false" publish_viz="false" />
-  <xacro:thermal_gazebo_sensor prefix_y="middle" publish_msg="false" publish_viz="false" />
-  <xacro:thermal_gazebo_sensor prefix_y="left" publish_msg="false" publish_viz="false" />
-  <xacro:thermal_gazebo_sensor prefix_y="right" publish_msg="false" publish_viz="false" />
-  <xacro:microphone_gazebo_sensor publish_msg="false" publish_viz="false" />
+  <xacro:sonar_gazebo_sensor name="linear" />
+  <xacro:sonar_gazebo_sensor name="left" />
+  <xacro:sonar_gazebo_sensor name="right" />
+  <xacro:co2_gazebo_sensor />
+  <xacro:thermal_gazebo_sensor prefix_y="middle" />
+  <xacro:thermal_gazebo_sensor prefix_y="left" />
+  <xacro:thermal_gazebo_sensor prefix_y="right" />
+  <xacro:microphone_gazebo_sensor />
 <!-- Load Transmissions ################################################### -->
   <xacro:wheel_transmission prefix_y="left" prefix_x="front" />

File: pandora_gazebo_description/urdf/gears/sensors/co2_sensor.gazebo.xacro (robot description, xacro)
@@ -2,6 +2,5 @@
 <robot xmlns:xacro="http://ros.org/wiki/xacro" >
 <!-- ###################################################################### -->
-  <xacro:macro name="co2_gazebo_sensor"
-               params="publish_msg publish_viz" >
+  <xacro:macro name="co2_gazebo_sensor" >
     <gazebo reference="co2_frame" >
       <sensor name="co2"
@@ -12,12 +11,6 @@
           <!--============================================================= -->
           <image>
-            <xacro:if value="${publish_viz}" >
-              <width>640</width>
-              <height>480</height>
-            </xacro:if>
-            <xacro:unless value="${publish_viz}" >
-              <width>8</width>
-              <height>8</height>
-            </xacro:unless>
+            <width>8</width>
+            <height>8</height>
           </image>
           <!--============================================================= -->
@@ -36,8 +29,4 @@
           <topicName>co2</topicName>
           <!--============================================================= -->
-          <publishMsg>${publish_msg}</publishMsg>
-          <!--============================================================= -->
-          <publishViz>${publish_viz}</publishViz>
-          <!--============================================================= -->
         </plugin>
         <!--=============================================================== -->

File: pandora_gazebo_description/urdf/gears/sensors/microphone_sensor.gazebo.xacro (robot description, xacro)
@@ -2,6 +2,5 @@
 <robot xmlns:xacro="http://ros.org/wiki/xacro" >
 <!-- ###################################################################### -->
-  <xacro:macro name="microphone_gazebo_sensor"
-               params="publish_msg publish_viz" >
+  <xacro:macro name="microphone_gazebo_sensor" >
     <gazebo reference="microphone_frame" >
       <sensor name="microphone"
@@ -12,12 +11,6 @@
           <!--============================================================= -->
           <image>
-            <xacro:if value="${publish_viz}" >
-              <width>640</width>
-              <height>480</height>
-            </xacro:if>
-            <xacro:unless value="${publish_viz}" >
-              <width>8</width>
-              <height>8</height>
-            </xacro:unless>
+            <width>8</width>
+            <height>8</height>
           </image>
           <!--============================================================= -->
@@ -36,8 +29,4 @@
           <topicName>sound</topicName>
           <!--============================================================= -->
-          <publishMsg>${publish_msg}</publishMsg>
-          <!--============================================================= -->
-          <publishViz>${publish_viz}</publishViz>
-          <!--============================================================= -->
         </plugin>
         <!--=============================================================== -->

File: pandora_gazebo_description/urdf/gears/sensors/sonar_sensor.gazebo.xacro (robot description, xacro)
@@ -3,5 +3,5 @@
 <!-- ###################################################################### -->
   <xacro:macro name="sonar_gazebo_sensor"
-               params="name publish_msg" >
+               params="name" >
     <gazebo reference="${name}_sonar_frame" >
       <sensor name="${name}_sonar"
@@ -44,6 +44,4 @@
           <gaussianNoise>0.0</gaussianNoise>
           <!--============================================================= -->
-          <publishMsg>${publish_msg}</publishMsg>
-          <!--============================================================= -->
         </plugin>
         <!--=============================================================== -->

File: pandora_gazebo_description/urdf/gears/sensors/thermal_sensor.gazebo.xacro (robot description, xacro)
@@ -3,5 +3,5 @@
 <!-- ###################################################################### -->
   <xacro:macro name="thermal_gazebo_sensor"
-               params="prefix_y publish_msg publish_viz" >
+               params="prefix_y" >
     <gazebo reference="${prefix_y}_thermal_frame" >
       <sensor name="${prefix_y}_thermal"
@@ -12,12 +12,6 @@
           <!--============================================================= -->
           <image>
-            <xacro:if value="${publish_viz}" >
-              <width>640</width>
-              <height>480</height>
-            </xacro:if>
-            <xacro:unless value="${publish_viz}" >
-              <width>8</width>
-              <height>8</height>
-            </xacro:unless>
+            <width>8</width>
+            <height>8</height>
           </image>
           <!--============================================================= -->
@@ -36,8 +30,4 @@
           <topicName>thermal</topicName>
           <!--============================================================= -->
-          <publishMsg>${publish_msg}</publishMsg>
-          <!--============================================================= -->
-          <publishViz>${publish_viz}</publishViz>
-          <!--============================================================= -->
         </plugin>
         <!--=============================================================== -->

File: pandora_gazebo_description/urdf/woody/sensors/sonar_sensor.gazebo.xacro (robot description, xacro)
@@ -3,5 +3,5 @@
 <!-- ###################################################################### -->
   <xacro:macro name="sonar_gazebo_sensor"
-               params="name publish_msg" >
+               params="name" >
     <gazebo reference="${name}_sonar_frame" >
       <sensor name="${name}_sonar"
@@ -45,6 +45,4 @@
           <gaussianNoise>0.0</gaussianNoise>
           <!--============================================================= -->
-          <publishMsg>${publish_msg}</publishMsg>
-          <!--============================================================= -->
         </plugin>
         <!--=============================================================== -->
