Commit message: Remove args to publish msg and viz from sensor plugins

File: pandora_gazebo_description/urdf/woody/woody.gazebo.xacro (robot description, xacro)
@@ -135,15 +135,5 @@
           <xacro:if value="${enable_left_sonar_sensor}" >
             <xacro:if value="${enable_left_sonar_gazebo_sensor}" >
-              <xacro:if value="$(arg control)" >
-                <xacro:if value="$(arg interface)" >
-                  <xacro:sonar_gazebo_sensor name="left" publish_msg="false" />
-                </xacro:if>
-                <xacro:unless value="$(arg interface)" >
-                  <xacro:sonar_gazebo_sensor name="left" publish_msg="true" />
-                </xacro:unless>
-              </xacro:if>
-              <xacro:unless value="$(arg control)" >
-                <xacro:sonar_gazebo_sensor name="left" publish_msg="true" />
-              </xacro:unless>
+              <xacro:sonar_gazebo_sensor name="left" />
             </xacro:if>
           </xacro:if>
@@ -151,15 +141,5 @@
           <xacro:if value="${enable_right_sonar_sensor}" >
             <xacro:if value="${enable_right_sonar_gazebo_sensor}" >
-              <xacro:if value="$(arg control)" >
-                <xacro:if value="$(arg interface)" >
-                  <xacro:sonar_gazebo_sensor name="right" publish_msg="false" />
-                </xacro:if>
-                <xacro:unless value="$(arg interface)" >
-                  <xacro:sonar_gazebo_sensor name="right" publish_msg="true" />
-                </xacro:unless>
-              </xacro:if>
-              <xacro:unless value="$(arg control)" >
-                <xacro:sonar_gazebo_sensor name="right" publish_msg="true" />
-              </xacro:unless>
+              <xacro:sonar_gazebo_sensor name="right" />
             </xacro:if>
           </xacro:if>
@@ -169,30 +149,5 @@
       <xacro:if value="${enable_co2_sensor}" >
         <xacro:if value="${enable_co2_gazebo_sensor}" >
-          <xacro:if value="$(arg control)" >
-            <xacro:if value="$(arg interface)" >
-              <xacro:if value="$(arg sensors_viz)" >
-                <xacro:co2_gazebo_sensor publish_msg="false" publish_viz="true" />
-              </xacro:if>
-              <xacro:unless value="$(arg sensors_viz)" >
-                <xacro:co2_gazebo_sensor publish_msg="false" publish_viz="false" />
-              </xacro:unless>
-            </xacro:if>
-            <xacro:unless value="$(arg interface)" >
-              <xacro:if value="$(arg sensors_viz)" >
-                <xacro:co2_gazebo_sensor publish_msg="true" publish_viz="true" />
-              </xacro:if>
-              <xacro:unless value="$(arg sensors_viz)" >
-                <xacro:co2_gazebo_sensor publish_msg="true" publish_viz="false" />
-              </xacro:unless>
-            </xacro:unless>
-          </xacro:if>
-          <xacro:unless value="$(arg control)" >
-            <xacro:if value="$(arg sensors_viz)" >
-              <xacro:co2_gazebo_sensor publish_msg="true" publish_viz="true" />
-            </xacro:if>
-            <xacro:unless value="$(arg sensors_viz)" >
-              <xacro:co2_gazebo_sensor publish_msg="true" publish_viz="false" />
-            </xacro:unless>
-          </xacro:unless>
+          <xacro:co2_gazebo_sensor />
         </xacro:if>
       </xacro:if>
@@ -200,30 +155,5 @@
         <xacro:if value="${enable_thermal_gazebo_sensor}" >
           <xacro:if value="${enable_thermal_gazebo_sensor}" >
-            <xacro:if value="$(arg control)" >
-              <xacro:if value="$(arg interface)" >
-                <xacro:if value="$(arg sensors_viz)" >
-                  <xacro:thermal_gazebo_sensor prefix_y="middle" publish_msg="false" publish_viz="true" />
-                </xacro:if>
-                <xacro:unless value="$(arg sensors_viz)" >
-                  <xacro:thermal_gazebo_sensor prefix_y="middle" publish_msg="false" publish_viz="false" />
-                </xacro:unless>
-              </xacro:if>
-              <xacro:unless value="$(arg interface)" >
-                <xacro:if value="$(arg sensors_viz)" >
-                  <xacro:thermal_gazebo_sensor prefix_y="middle" publish_msg="true" publish_viz="true" />
-                </xacro:if>
-                <xacro:unless value="$(arg sensors_viz)" >
-                  <xacro:thermal_gazebo_sensor prefix_y="middle" publish_msg="true" publish_viz="false" />
-                </xacro:unless>
-              </xacro:unless>
-            </xacro:if>
-            <xacro:unless value="$(arg control)" >
-              <xacro:if value="$(arg sensors_viz)" >
-                <xacro:thermal_gazebo_sensor prefix_y="middle" publish_msg="true" publish_viz="true" />
-              </xacro:if>
-              <xacro:unless value="$(arg sensors_viz)" >
-                <xacro:thermal_gazebo_sensor prefix_y="middle" publish_msg="true" publish_viz="false" />
-              </xacro:unless>
-            </xacro:unless>
+            <xacro:thermal_gazebo_sensor prefix_y="middle" />
           </xacro:if>
         </xacro:if>
@@ -231,30 +161,5 @@
       <xacro:if value="${enable_microphone_sensor}" >
         <xacro:if value="${enable_microphone_gazebo_sensor}" >
-          <xacro:if value="$(arg control)" >
-            <xacro:if value="$(arg interface)" >
-              <xacro:if value="$(arg sensors_viz)" >
-                <xacro:microphone_gazebo_sensor publish_msg="false" publish_viz="true" />
-              </xacro:if>
-              <xacro:unless value="$(arg sensors_viz)" >
-                <xacro:microphone_gazebo_sensor publish_msg="false" publish_viz="false" />
-              </xacro:unless>
-            </xacro:if>
-            <xacro:unless value="$(arg interface)" >
-              <xacro:if value="$(arg sensors_viz)" >
-                <xacro:microphone_gazebo_sensor publish_msg="true" publish_viz="true" />
-              </xacro:if>
-              <xacro:unless value="$(arg sensors_viz)" >
-                <xacro:microphone_gazebo_sensor publish_msg="true" publish_viz="false" />
-              </xacro:unless>
-            </xacro:unless>
-          </xacro:if>
-          <xacro:unless value="$(arg control)" >
-            <xacro:if value="$(arg sensors_viz)" >
-              <xacro:microphone_gazebo_sensor publish_msg="true" publish_viz="true" />
-            </xacro:if>
-            <xacro:unless value="$(arg sensors_viz)" >
-              <xacro:microphone_gazebo_sensor publish_msg="true" publish_viz="false" />
-            </xacro:unless>
-          </xacro:unless>
+          <xacro:microphone_gazebo_sensor />
         </xacro:if>
       </xacro:if>

File: pandora_gazebo_description/urdf/woody/woody_simplified.gazebo.xacro (robot description, xacro)
@@ -43,10 +43,10 @@
 <!--  <xacro:camera_gazebo_sensor prefix_y="left" />-->
 <!--  <xacro:camera_gazebo_sensor prefix_y="right" />-->
-  <xacro:sonar_gazebo_sensor name="left" publish_msg="false" />
-  <xacro:sonar_gazebo_sensor name="right" publish_msg="false" />
-<!--  TODO: <xacro:flir_gazebo_sensor publish_msg="false" publish_viz="false" />-->
-<xacro:co2_gazebo_sensor publish_msg="true" publish_viz="false" />
-<xacro:thermal_gazebo_sensor prefix_y="middle" publish_msg="true" publish_viz="false" />
-<!--  <xacro:microphone_gazebo_sensor publish_msg="false" publish_viz="false" />-->
+  <xacro:sonar_gazebo_sensor name="left" />
+  <xacro:sonar_gazebo_sensor name="right" />
+<!--  TODO: <xacro:flir_gazebo_sensor />-->
+  <xacro:co2_gazebo_sensor />
+  <xacro:thermal_gazebo_sensor prefix_y="middle" />
+<!--  <xacro:microphone_gazebo_sensor />-->
 <!-- Load Transmissions ################################################### -->
   <xacro:wheel_transmission prefix_y="left" prefix_x="front" />
