Commit message: Remove unused elements from description [ci skip]

File: pandora_gazebo_description/urdf/woody/plugins/ros_skid_steer_drive_plugin.gazebo.xacro (robot description, xacro)
@@ -16,5 +16,5 @@
         <rightRearJoint>right_rear_wheel_joint</rightRearJoint>
         <!-- ============================================================== -->
-        <wheelSeparation>${wheel_separation}</wheelSeparation>
+        <wheelSeparation>${track}</wheelSeparation>
         <wheelDiameter>${ 2 * wheel_radius }</wheelDiameter>
         <!-- ============================================================== -->

File: pandora_gazebo_description/urdf/woody/sdf_configurations.xacro (robot description, xacro)
@@ -10,5 +10,5 @@
   <!-- ==================================================================== -->
   <!-- Sensors ============================================================ -->
-  <xacro:property name="enable_gazebo_sensors" value="true" />
+  <xacro:property name="enable_gazebo_sensors" value="false" />
     <!-- ================================================================== -->
     <xacro:property name="enable_laser_gazebo_sensor" value="true" />
@@ -16,21 +16,17 @@
     <xacro:property name="enable_kinect_gazebo_sensor" value="true" />
     <!-- ================================================================== -->
-    <xacro:property name="enable_camera_gazebo_sensors" value="true" />
+    <xacro:property name="enable_camera_gazebo_sensors" value="false" />
       <xacro:property name="enable_left_camera_gazebo_sensor" value="true" />
       <xacro:property name="enable_right_camera_gazebo_sensor" value="true" />
     <!-- ================================================================== -->
-    <xacro:property name="enable_sonar_gazebo_sensors" value="true" />
-      <xacro:property name="enable_linear_sonar_gazebo_sensor" value="true" />
+    <xacro:property name="enable_sonar_gazebo_sensors" value="false" />
       <xacro:property name="enable_left_sonar_gazebo_sensor" value="true" />
       <xacro:property name="enable_right_sonar_gazebo_sensor" value="true" />
     <!-- ================================================================== -->
-    <xacro:property name="enable_thermal_gazebo_sensors" value="true" />
-      <xacro:property name="enable_middle_thermal_gazebo_sensor" value="true" />
-      <xacro:property name="enable_left_thermal_gazebo_sensor" value="true" />
-      <xacro:property name="enable_right_thermal_gazebo_sensor" value="true" />
+    <xacro:property name="enable_thermal_gazebo_sensor" value="false" />
     <!-- ================================================================== -->
-    <xacro:property name="enable_co2_gazebo_sensor" value="true" />
+    <xacro:property name="enable_co2_gazebo_sensor" value="false" />
     <!-- ================================================================== -->
-    <xacro:property name="enable_microphone_gazebo_sensor" value="true" />
+    <xacro:property name="enable_microphone_gazebo_sensor" value="false" />
   <!-- ==================================================================== -->
   <!-- Physics ============================================================ -->
@@ -43,9 +39,4 @@
     <!-- ================================================================== -->
     <xacro:property name="enable_wheel_joint_physics" value="false" />
-    <!-- ================================================================== -->
-    <xacro:property name="enable_linear_elevator_joint_physics" value="true" />
-    <!-- ================================================================== -->
-    <xacro:property name="enable_linear_head_yaw_joint_physics" value="false" />
-    <xacro:property name="enable_linear_head_pitch_joint_physics" value="false" />
     <!-- ================================================================== -->
     <xacro:property name="enable_laser_roll_joint_physics" value="false" />
@@ -60,9 +51,9 @@
     <xacro:property name="enable_pandora_differential_plugin" value="true" />
     <!-- ================================================================== -->
-    <xacro:property name="enable_pandora_p3d_plugin" value="true" />
+    <xacro:property name="enable_pandora_p3d_plugin" value="false" />
     <!-- ================================================================== -->
-    <xacro:property name="enable_pandora_imu_stabilizer_plugin" value="true" />
+    <xacro:property name="enable_pandora_imu_stabilizer_plugin" value="false" />
     <!-- ================================================================== -->
-    <xacro:property name="enable_ros_imu_plugin" value="true" />
+    <xacro:property name="enable_ros_imu_plugin" value="false" />
     <!-- ================================================================== -->
     <xacro:property name="enable_ros_skid_steer_drive_plugin" value="true" />
@@ -70,10 +61,10 @@
 <!-- Joint Physics ######################################################## -->
   <!-- Wheels ============================================================= -->
-  <xacro:property name="wheel_mu_1" value="0.85" />
-  <xacro:property name="wheel_mu_2" value="0.85" />
-  <xacro:property name="wheel_k_p" value="10000000.0" />
+  <xacro:property name="wheel_mu_1" value="0.5" /> <!-- FIXME -->
+  <xacro:property name="wheel_mu_2" value="0.5" /> <!-- FIXME -->
+  <xacro:property name="wheel_k_p" value="1000000.0" />
   <xacro:property name="wheel_k_d" value="1.0" />
-  <xacro:property name="wheel_min_depth" value="0.0001" />
-  <xacro:property name="wheel_max_contacts" value="1" />
+  <xacro:property name="wheel_min_depth" value="0.001" />
+  <xacro:property name="wheel_max_contacts" value="10" />
   <!-- ==================================================================== -->
 <!-- Plugin Parameters #################################################### -->

File: pandora_gazebo_description/urdf/woody/woody.gazebo.xacro (robot description, xacro)
@@ -14,7 +14,4 @@
   <xacro:include filename="$(find pandora_gazebo_description)/urdf/woody/physics/side_joint_physics.gazebo.xacro" />
   <xacro:include filename="$(find pandora_gazebo_description)/urdf/woody/physics/wheel_joint_physics.gazebo.xacro" />
-  <xacro:include filename="$(find pandora_gazebo_description)/urdf/woody/physics/linear_elevator_joint_physics.gazebo.xacro" />
-  <xacro:include filename="$(find pandora_gazebo_description)/urdf/woody/physics/linear_head_pitch_joint_physics.gazebo.xacro" />
-  <xacro:include filename="$(find pandora_gazebo_description)/urdf/woody/physics/linear_head_yaw_joint_physics.gazebo.xacro" />
   <xacro:include filename="$(find pandora_gazebo_description)/urdf/woody/physics/laser_roll_joint_physics.gazebo.xacro" />
   <xacro:include filename="$(find pandora_gazebo_description)/urdf/woody/physics/laser_pitch_joint_physics.gazebo.xacro" />
@@ -31,6 +28,4 @@
   <!-- ==================================================================== -->
   <xacro:include filename="$(find pandora_gazebo_description)/urdf/woody/transmissions/wheel_transmission.xacro" />
-  <xacro:include filename="$(find pandora_gazebo_description)/urdf/woody/transmissions/linear_elevator_transmission.xacro" />
-  <xacro:include filename="$(find pandora_gazebo_description)/urdf/woody/transmissions/linear_head_transmission.xacro" />
   <xacro:include filename="$(find pandora_gazebo_description)/urdf/woody/transmissions/laser_sensor_transmission.xacro" />
   <xacro:include filename="$(find pandora_gazebo_description)/urdf/woody/transmissions/kinect_sensor_transmission.xacro" />
@@ -75,17 +70,4 @@
     </xacro:if>
     <!-- ================================================================ -->
-    <!-- ================================================================ -->
-    <xacro:if value="${enable_linear_elevator_joint_physics}" >
-      <xacro:linear_elevator_joint_physics />
-    </xacro:if>
-    <!-- ================================================================ -->
-    <xacro:if value="${enable_linear_head_yaw_joint_physics}" >
-      <xacro:linear_head_yaw_joint_physics />
-    </xacro:if>
-    <!-- ================================================================ -->
-    <xacro:if value="${enable_linear_head_pitch_joint_physics}" >
-      <xacro:linear_head_pitch_joint_physics />
-    </xacro:if>
-    <!-- ================================================================ -->
     <xacro:if value="${enable_sensors}" >
       <!-- ================================================================ -->
@@ -148,20 +130,4 @@
       <xacro:if value="${enable_sonar_sensors}" >
         <xacro:if value="${enable_sonar_gazebo_sensors}" >
-          <!-- ============================================================ -->
-          <xacro:if value="${enable_linear_sonar_sensor}" >
-            <xacro:if value="${enable_linear_sonar_gazebo_sensor}" >
-              <xacro:if value="$(arg control)" >
-                <xacro:if value="$(arg interface)" >
-                  <xacro:sonar_gazebo_sensor name="linear" publish_msg="false" />
-                </xacro:if>
-                <xacro:unless value="$(arg interface)" >
-                  <xacro:sonar_gazebo_sensor name="linear" publish_msg="true" />
-                </xacro:unless>
-              </xacro:if>
-              <xacro:unless value="$(arg control)" >
-                <xacro:sonar_gazebo_sensor name="linear" publish_msg="true" />
-              </xacro:unless>
-            </xacro:if>
-          </xacro:if>
           <!-- ============================================================ -->
           <xacro:if value="${enable_left_sonar_sensor}" >
@@ -230,27 +196,16 @@
       </xacro:if>
       <xacro:if value="${enable_thermal_sensors}" >
-        <xacro:if value="${enable_thermal_gazebo_sensors}" >
-          <!-- ============================================================ -->
-          <xacro:if value="${enable_middle_thermal_sensor}" >
-            <xacro:if value="${enable_middle_thermal_gazebo_sensor}" >
-              <xacro:if value="$(arg control)" >
-                <xacro:if value="$(arg interface)" >
-                  <xacro:if value="$(arg sensors_viz)" >
-                    <xacro:thermal_gazebo_sensor prefix_y="middle" publish_msg="false" publish_viz="true" />
-                  </xacro:if>
-                  <xacro:unless value="$(arg sensors_viz)" >
-                    <xacro:thermal_gazebo_sensor prefix_y="middle" publish_msg="false" publish_viz="false" />
-                  </xacro:unless>
+        <xacro:if value="${enable_thermal_gazebo_sensor}" >
+          <xacro:if value="${enable_thermal_gazebo_sensor}" >
+            <xacro:if value="$(arg control)" >
+              <xacro:if value="$(arg interface)" >
+                <xacro:if value="$(arg sensors_viz)" >
+                  <xacro:thermal_gazebo_sensor prefix_y="middle" publish_msg="false" publish_viz="true" />
                 </xacro:if>
-                <xacro:unless value="$(arg interface)" >
-                  <xacro:if value="$(arg sensors_viz)" >
-                    <xacro:thermal_gazebo_sensor prefix_y="middle" publish_msg="true" publish_viz="true" />
-                  </xacro:if>
-                  <xacro:unless value="$(arg sensors_viz)" >
-                    <xacro:thermal_gazebo_sensor prefix_y="middle" publish_msg="true" publish_viz="false" />
-                  </xacro:unless>
+                <xacro:unless value="$(arg sensors_viz)" >
+                  <xacro:thermal_gazebo_sensor prefix_y="middle" publish_msg="false" publish_viz="false" />
                 </xacro:unless>
               </xacro:if>
-              <xacro:unless value="$(arg control)" >
+              <xacro:unless value="$(arg interface)" >
                 <xacro:if value="$(arg sensors_viz)" >
                   <xacro:thermal_gazebo_sensor prefix_y="middle" publish_msg="true" publish_viz="true" />
@@ -261,68 +216,13 @@
               </xacro:unless>
             </xacro:if>
-          </xacro:if>
-          <!-- ============================================================ -->
-          <xacro:if value="${enable_left_thermal_sensor}" >
-            <xacro:if value="${enable_left_thermal_gazebo_sensor}" >
-              <xacro:if value="$(arg control)" >
-                <xacro:if value="$(arg interface)" >
-                  <xacro:if value="$(arg sensors_viz)" >
-                    <xacro:thermal_gazebo_sensor prefix_y="left" publish_msg="false" publish_viz="true" />
-                  </xacro:if>
-                  <xacro:unless value="$(arg sensors_viz)" >
-                    <xacro:thermal_gazebo_sensor prefix_y="left" publish_msg="false" publish_viz="false" />
-                  </xacro:unless>
-                </xacro:if>
-                <xacro:unless value="$(arg interface)" >
-                  <xacro:if value="$(arg sensors_viz)" >
-                    <xacro:thermal_gazebo_sensor prefix_y="left" publish_msg="true" publish_viz="true" />
-                  </xacro:if>
-                  <xacro:unless value="$(arg sensors_viz)" >
-                    <xacro:thermal_gazebo_sensor prefix_y="left" publish_msg="true" publish_viz="false" />
-                  </xacro:unless>
-                </xacro:unless>
-              </xacro:if>
-              <xacro:unless value="$(arg control)" >
-                <xacro:if value="$(arg sensors_viz)" >
-                  <xacro:thermal_gazebo_sensor prefix_y="left" publish_msg="true" publish_viz="true" />
-                </xacro:if>
-                <xacro:unless value="$(arg sensors_viz)" >
-                  <xacro:thermal_gazebo_sensor prefix_y="left" publish_msg="true" publish_viz="false" />
-                </xacro:unless>
-              </xacro:unless>
-            </xacro:if>
-          </xacro:if>
-          <!-- ============================================================ -->
-          <xacro:if value="${enable_right_thermal_sensor}" >
-            <xacro:if value="${enable_right_thermal_gazebo_sensor}" >
-              <xacro:if value="$(arg control)" >
-                <xacro:if value="$(arg interface)" >
-                  <xacro:if value="$(arg sensors_viz)" >
-                    <xacro:thermal_gazebo_sensor prefix_y="right" publish_msg="false" publish_viz="true" />
-                  </xacro:if>
-                  <xacro:unless value="$(arg sensors_viz)" >
-                    <xacro:thermal_gazebo_sensor prefix_y="right" publish_msg="false" publish_viz="false" />
-                  </xacro:unless>
-                </xacro:if>
-                <xacro:unless value="$(arg interface)" >
-                  <xacro:if value="$(arg sensors_viz)" >
-                    <xacro:thermal_gazebo_sensor prefix_y="right" publish_msg="true" publish_viz="true" />
-                  </xacro:if>
-                  <xacro:unless value="$(arg sensors_viz)" >
-                    <xacro:thermal_gazebo_sensor prefix_y="right" publish_msg="true" publish_viz="false" />
-                  </xacro:unless>
-                </xacro:unless>
-              </xacro:if>
-              <xacro:unless value="$(arg control)" >
-                <xacro:if value="$(arg sensors_viz)" >
-                  <xacro:thermal_gazebo_sensor prefix_y="right" publish_msg="true" publish_viz="true" />
-                </xacro:if>
-                <xacro:unless value="$(arg sensors_viz)" >
-                  <xacro:thermal_gazebo_sensor prefix_y="right" publish_msg="true" publish_viz="false" />
-                </xacro:unless>
-              </xacro:unless>
-            </xacro:if>
-          </xacro:if>
-          <!-- ============================================================ -->
+            <xacro:unless value="$(arg control)" >
+              <xacro:if value="$(arg sensors_viz)" >
+                <xacro:thermal_gazebo_sensor prefix_y="middle" publish_msg="true" publish_viz="true" />
+              </xacro:if>
+              <xacro:unless value="$(arg sensors_viz)" >
+                <xacro:thermal_gazebo_sensor prefix_y="middle" publish_msg="true" publish_viz="false" />
+              </xacro:unless>
+            </xacro:unless>
+          </xacro:if>
         </xacro:if>
       </xacro:if>
@@ -365,7 +265,4 @@
     <xacro:wheel_transmission prefix_y="right" prefix_x="front" />
     <xacro:wheel_transmission prefix_y="right" prefix_x="rear" />
-    <xacro:linear_elevator_transmission />
-    <xacro:linear_head_transmission rotation="pitch" />
-    <xacro:linear_head_transmission rotation="yaw" />
     <xacro:if value="${enable_sensors}" >
       <!-- ================================================================ -->

File: pandora_gazebo_description/urdf/woody/woody_simplified.gazebo.xacro (robot description, xacro)
@@ -5,5 +5,4 @@
   <xacro:include filename="$(find pandora_robots_description)/urdf/woody/woody.urdf.xacro" />
   <xacro:include filename="$(find pandora_gazebo_description)/urdf/woody/physics/wheel_link_physics.gazebo.xacro" />
-  <xacro:include filename="$(find pandora_gazebo_description)/urdf/woody/physics/linear_elevator_joint_physics.gazebo.xacro" />
   <xacro:include filename="$(find pandora_gazebo_description)/urdf/woody/sensors/laser_sensor.gazebo.xacro" />
   <xacro:include filename="$(find pandora_gazebo_description)/urdf/woody/sensors/kinect_sensor.gazebo.xacro" />
@@ -14,6 +13,4 @@
   <xacro:include filename="$(find pandora_gazebo_description)/urdf/woody/sensors/microphone_sensor.gazebo.xacro" />
   <xacro:include filename="$(find pandora_gazebo_description)/urdf/woody/transmissions/wheel_transmission.xacro" />
-  <xacro:include filename="$(find pandora_gazebo_description)/urdf/woody/transmissions/linear_elevator_transmission.xacro" />
-  <xacro:include filename="$(find pandora_gazebo_description)/urdf/woody/transmissions/linear_head_transmission.xacro" />
   <xacro:include filename="$(find pandora_gazebo_description)/urdf/woody/transmissions/laser_sensor_transmission.xacro" />
   <xacro:include filename="$(find pandora_gazebo_description)/urdf/woody/transmissions/kinect_sensor_transmission.xacro" />
@@ -37,6 +34,6 @@
   <xacro:wheel_link_physics prefix_y="right" prefix_x="front" />
   <xacro:wheel_link_physics prefix_y="right" prefix_x="rear" />
-  <xacro:linear_elevator_joint_physics />
 <!-- Load Gazebo Sensors ################################################## -->
+  <!--
   <xacro:laser_gazebo_sensor />
   <xacro:kinect_gazebo_sensor />
@@ -48,24 +45,24 @@
   <xacro:co2_gazebo_sensor publish_msg="false" publish_viz="false" />
   <xacro:thermal_gazebo_sensor prefix_y="middle" publish_msg="false" publish_viz="false" />
-  <xacro:thermal_gazebo_sensor prefix_y="left" publish_msg="false" publish_viz="false" />
-  <xacro:thermal_gazebo_sensor prefix_y="right" publish_msg="false" publish_viz="false" />
   <xacro:microphone_gazebo_sensor publish_msg="false" publish_viz="false" />
+  -->
 <!-- Load Transmissions ################################################### -->
+  <!--
   <xacro:wheel_transmission prefix_y="left" prefix_x="front" />
   <xacro:wheel_transmission prefix_y="left" prefix_x="rear" />
   <xacro:wheel_transmission prefix_y="right" prefix_x="front" />
   <xacro:wheel_transmission prefix_y="right" prefix_x="rear" />
-  <xacro:linear_elevator_transmission />
-  <xacro:linear_head_transmission rotation="yaw" />
-  <xacro:linear_head_transmission rotation="pitch" />
   <xacro:laser_sensor_transmission rotation="roll" />
   <xacro:laser_sensor_transmission rotation="pitch" />
   <xacro:kinect_sensor_transmission rotation="pitch" />
   <xacro:kinect_sensor_transmission rotation="yaw" />
+  -->
 <!-- Load Plugins ######################################################### -->
-  <xacro:pandora_differential_plugin publish_joint_states="false" />
-  <xacro:pandora_p3d_plugin />
-  <xacro:gazebo_ros_control_plugin namespace="/"
-                                   hardware_interface="pandora_gazebo_interface/GazeboInterface" />
+  <xacro:ros_skid_steer_drive_plugin />
+  <xacro:pandora_differential_plugin publish_joint_states="true" />
+  <!-- <xacro:pandora_differential_plugin publish_joint_states="false" /> -->
+  <!-- <xacro:pandora_p3d_plugin /> -->
+  <!-- <xacro:gazebo_ros_control_plugin namespace="/"
+                                   hardware_interface="pandora_gazebo_interface/GazeboInterface" /> -->
 <!-- ###################################################################### -->
 </robot>
