Commit message: Update launchers [ci skip]

File: pandora_gazebo_description/urdf/woody/sdf_configurations.xacro (robot description, xacro)
@@ -61,6 +61,6 @@
 <!-- Joint Physics ######################################################## -->
   <!-- Wheels ============================================================= -->
-  <xacro:property name="wheel_mu_1" value="0.5" /> <!-- FIXME -->
-  <xacro:property name="wheel_mu_2" value="0.5" /> <!-- FIXME -->
+  <xacro:property name="wheel_mu_1" value="0.75" /> <!-- FIXME -->
+  <xacro:property name="wheel_mu_2" value="0.75" /> <!-- FIXME -->
   <xacro:property name="wheel_k_p" value="1000000.0" />
   <xacro:property name="wheel_k_d" value="1.0" />

File: pandora_gazebo_description/urdf/woody/woody_simplified.gazebo.xacro (robot description, xacro)
@@ -28,5 +28,6 @@
   <xacro:property name="wheel_max_contacts" value="10" />
 <!-- Load URDF ############################################################ -->
-  <xacro:woody_urdf fixed="false" />
+  <xacro:woody_urdf fixed="true" />
+  <!-- <xacro:woody_urdf fixed="false" /> -->
 <!-- Load Physics ######################################################### -->
   <xacro:wheel_link_physics prefix_y="left" prefix_x="front" />

Commit message: Add temp properties at sdf_configurations to bringup non-simplified woody description

File: pandora_gazebo_description/urdf/woody/sdf_configurations.xacro (robot description, xacro)
@@ -9,5 +9,19 @@
   <xacro:property name="static_robot" value="false" />
   <!-- ==================================================================== -->
-  <!-- Sensors ============================================================ -->
+  <!-- Model Sensors ====================================================== -->
+   <!-- FIXME: Remove all model properties (should be set in URDF) -->
+  <xacro:property name="enable_sensors" value="true" />
+    <xacro:property name="enable_laser_sensor" value="true" />
+    <xacro:property name="enable_kinect_sensor" value="true" />
+    <xacro:property name="enable_camera_sensors" value="true" />
+      <xacro:property name="enable_left_camera_sensor" value="true" />
+      <xacro:property name="enable_right_camera_sensor" value="true" />
+    <xacro:property name="enable_sonar_sensors" value="true" />
+      <xacro:property name="enable_left_sonar_sensor" value="true" />
+      <xacro:property name="enable_right_sonar_sensor" value="true" />
+    <xacro:property name="enable_thermal_sensor" value="true" />
+    <xacro:property name="enable_co2_sensor" value="true" />
+    <xacro:property name="enable_microphone_sensor" value="false" />
+  <!-- Gazebo Sensors ===================================================== -->
   <xacro:property name="enable_gazebo_sensors" value="true" />
     <!-- ================================================================== -->

File: pandora_gazebo_description/urdf/woody/woody.gazebo.xacro (robot description, xacro)
@@ -152,5 +152,5 @@
         </xacro:if>
       </xacro:if>
-      <xacro:if value="${enable_thermal_sensors}" >
+      <xacro:if value="${enable_thermal_sensor}" >
         <xacro:if value="${enable_thermal_gazebo_sensor}" >
           <xacro:if value="${enable_thermal_gazebo_sensor}" >
@@ -233,5 +233,5 @@
     <xacro:if value="$(arg interface)" >
       <xacro:gazebo_ros_control_plugin namespace="/"
-                                       hardware_interface="pandora_gazebo_interface/GazeboInterface" />
+                                       hardware_interface="pandora_gazebo_interface/WoodyGazeboInterface" />
     </xacro:if>
     <xacro:unless value="$(arg interface)" >

Commit message: Remove thermal gazebo sensor from woody

File: pandora_gazebo_description/urdf/woody/sdf_configurations.xacro (robot description, xacro)
@@ -20,5 +20,5 @@
       <xacro:property name="enable_left_sonar_sensor" value="true" />
       <xacro:property name="enable_right_sonar_sensor" value="true" />
-    <xacro:property name="enable_thermal_sensor" value="true" />
+    <xacro:property name="enable_thermal_sensor" value="false" />
     <xacro:property name="enable_co2_sensor" value="true" />
     <xacro:property name="enable_microphone_sensor" value="false" />
@@ -38,5 +38,5 @@
       <xacro:property name="enable_right_sonar_gazebo_sensor" value="true" />
     <!-- ================================================================== -->
-    <xacro:property name="enable_thermal_gazebo_sensor" value="true" />
+    <xacro:property name="enable_thermal_gazebo_sensor" value="false" />
     <!-- ================================================================== -->
     <xacro:property name="enable_co2_gazebo_sensor" value="true" />

File: pandora_gazebo_description/urdf/woody/woody_simplified.gazebo.xacro (robot description, xacro)
@@ -45,8 +45,6 @@
   <xacro:sonar_gazebo_sensor name="left" />
   <xacro:sonar_gazebo_sensor name="right" />
-<!--  TODO: <xacro:flir_gazebo_sensor />-->
+<!--  <xacro:flir_gazebo_sensor />--> <!-- TODO -->
   <xacro:co2_gazebo_sensor />
-  <xacro:thermal_gazebo_sensor prefix_y="middle" />
-<!--  <xacro:microphone_gazebo_sensor />-->
 <!-- Load Transmissions ################################################### -->
   <xacro:wheel_transmission prefix_y="left" prefix_x="front" />
