Commit message: Remap gears' sensor topic names

File: pandora_gazebo_description/urdf/gears/sensors/co2_sensor.gazebo.xacro (robot description, xacro)
@@ -30,8 +30,9 @@
         <plugin name="co2ros"
                 filename="libpandora_gazebo_plugins_pandora_co2_plugin.so" >
+          <robotNamespace>gazebo_sensors</robotNamespace>
           <!--============================================================= -->
           <frameName>co2_frame</frameName>
           <!--============================================================= -->
-          <topicName>sensors/co2</topicName>
+          <topicName>co2</topicName>
           <!--============================================================= -->
           <publishMsg>${publish_msg}</publishMsg>

File: pandora_gazebo_description/urdf/gears/sensors/microphone_sensor.gazebo.xacro (robot description, xacro)
@@ -30,8 +30,9 @@
         <plugin name="microphone2ros"
                 filename="libpandora_gazebo_plugins_pandora_microphone_plugin.so" >
+          <robotNamespace>gazebo_sensors</robotNamespace>
           <!--============================================================= -->
           <frameName>microphone_frame</frameName>
           <!--============================================================= -->
-          <topicName>sensors/sound</topicName>
+          <topicName>sound</topicName>
           <!--============================================================= -->
           <publishMsg>${publish_msg}</publishMsg>

File: pandora_gazebo_description/urdf/gears/sensors/sonar_sensor.gazebo.xacro (robot description, xacro)
@@ -36,10 +36,9 @@
         <plugin name="sonar2ros"
                 filename="libpandora_gazebo_plugins_pandora_sonar_plugin.so" >
-          <!--============================================================= -->
-          <robotNamespace></robotNamespace>
+          <robotNamespace>gazebo_sensors</robotNamespace>
           <!--============================================================= -->
           <frameName>${name}_sonar_frame</frameName>
           <!--============================================================= -->
-          <topicName>/sensors/sonar</topicName> <!-- FIXME -->
+          <topicName>sonar</topicName> <!-- FIXME -->
           <!--============================================================= -->
           <gaussianNoise>0.0</gaussianNoise>

File: pandora_gazebo_description/urdf/gears/sensors/thermal_sensor.gazebo.xacro (robot description, xacro)
@@ -30,8 +30,9 @@
         <plugin name="thermal2ros"
                 filename="libpandora_gazebo_plugins_pandora_thermal_plugin.so" >
+          <robotNamespace>gazebo_sensors</robotNamespace>
           <!--============================================================= -->
           <frameName>${prefix_y}_thermal_optical_frame</frameName>
           <!--============================================================= -->
-          <topicName>sensors/thermal</topicName>
+          <topicName>thermal</topicName>
           <!--============================================================= -->
           <publishMsg>${publish_msg}</publishMsg>

File: pandora_gazebo_description/urdf/woody/sensors/co2_sensor.gazebo.xacro (robot description, xacro)
@@ -34,5 +34,5 @@
           <frameName>co2_frame</frameName>
           <!--============================================================= -->
-          <topicName>sensors/co2</topicName>
+          <topicName>co2</topicName>
           <!--============================================================= -->
           <publishMsg>${publish_msg}</publishMsg>

File: pandora_gazebo_description/urdf/woody/sensors/microphone_sensor.gazebo.xacro (robot description, xacro)
@@ -34,5 +34,5 @@
           <frameName>microphone_frame</frameName>
           <!--============================================================= -->
-          <topicName>sensors/sound</topicName>
+          <topicName>sound</topicName>
           <!--============================================================= -->
           <publishMsg>${publish_msg}</publishMsg>

File: pandora_gazebo_description/urdf/woody/sensors/sonar_sensor.gazebo.xacro (robot description, xacro)
@@ -41,5 +41,5 @@
           <frameName>${name}_sonar_frame</frameName>
           <!--============================================================= -->
-          <topicName>sensors/sonar</topicName> <!-- FIXME -->
+          <topicName>sonar</topicName> <!-- FIXME -->
           <!--============================================================= -->
           <gaussianNoise>0.0</gaussianNoise>

File: pandora_gazebo_description/urdf/woody/sensors/thermal_sensor.gazebo.xacro (robot description, xacro)
@@ -34,5 +34,5 @@
           <frameName>${prefix_y}_thermal_optical_frame</frameName>
           <!--============================================================= -->
-          <topicName>sensors/thermal</topicName>
+          <topicName>thermal</topicName>
           <!--============================================================= -->
           <publishMsg>${publish_msg}</publishMsg>

File: pandora_gazebo_description/urdf/woody/woody_simplified.gazebo.xacro (robot description, xacro)
@@ -59,16 +59,10 @@
   <xacro:kinect_sensor_transmission rotation="pitch" />
 <!-- Load Plugins ######################################################### -->
-  <xacro:ros_skid_steer_drive_plugin />
-  <xacro:property name="wheel_joint_max_torque" value="50" />
-  <xacro:pandora_differential_plugin publish_joint_states="true" />
-<!-- <xacro:pandora_differential_plugin publish_joint_states="false" /> -->
-  <xacro:pandora_imu_stabilizer_plugin />
-<!-- <xacro:pandora_p3d_plugin /> -->
-<!--  <xacro:gazebo_ros_control_plugin namespace="/"-->
-<!--                                   hardware_interface="gazebo_ros_control/DefaultRobotHWSim" />-->
+  <xacro:pandora_differential_plugin publish_joint_states="false" />
+  <xacro:pandora_p3d_plugin />
   <xacro:gazebo_ros_control_plugin namespace="/"
-                                   hardware_interface="pandora_gazebo_interface/WoodyGazeboInterface" /> -->
-<!-- <xacro:pandora_wheel_physics_plugin/> -->
-<!-- <xacro:pandora_fdir_plugin />-->
+                                   hardware_interface="pandora_gazebo_interface/WoodyGazeboInterface" />
+<!--  <xacro:pandora_wheel_physics_plugin/> -->
+<!--  <xacro:pandora_fdir_plugin />-->
 <!-- ###################################################################### -->
 </robot>
