Commit message: Make robots and gazebo_sensors parent dirs of pandora_gazebo_description package

File: pandora_gazebo_description/woody/gazebo_urdf/plugins/pandora_differential_plugin.gazebo.xacro (robot description, xacro)
@@ -2,6 +2,5 @@
 <robot xmlns:xacro="http://ros.org/wiki/xacro" >
 <!-- ###################################################################### -->
-  <xacro:macro name="pandora_differential_plugin"
-               params="publish_joint_states" >
+  <xacro:macro name="pandora_differential_plugin" >
     <gazebo>
       <plugin name="PandoraDifferantialPlugin"
@@ -10,5 +9,5 @@
         <robotNamespace>${robot_namespace}</robotNamespace>
         <!-- ============================================================== -->
-        <publishJointStates>${publish_joint_states}</publishJointStates>
+        <publishJointStates>false</publishJointStates>
         <!-- ============================================================== -->
         <baseLink>base_link</baseLink>
