Commit message: Remove woody simplified gazebo urdf

File: pandora_gazebo_description/woody/gazebo_urdf/plugins/ros_skid_steer_drive_plugin.gazebo.xacro (robot description, xacro)
@@ -7,5 +7,5 @@
               filename="libgazebo_ros_skid_steer_drive.so" >
         <!-- ============================================================== -->
-        <robotNamespace>${robot_namespace}</robotNamespace>
+        <robotNamespace>/</robotNamespace>
         <!-- ============================================================== -->
         <updateRate>100.0</updateRate>
@@ -19,5 +19,5 @@
         <wheelDiameter>${ 2 * wheel_radius }</wheelDiameter>
         <!-- ============================================================== -->
-        <torque>${wheel_joint_max_torque}</torque>
+        <torque>50</torque>
         <!-- ============================================================== -->
         <robotBaseFrame>base_link</robotBaseFrame>

File: pandora_gazebo_description/woody/gazebo_urdf/sdf_configurations.xacro (robot description, xacro)
@@ -17,5 +17,3 @@
   <xacro:property name="wheel_min_depth" value="0.001" />
   <xacro:property name="wheel_max_contacts" value="10" />
-  <!-- Skid steer drive plugin parameters -->
-  <xacro:property name="wheel_joint_max_torque" value="50" />
 </robot>

File: pandora_gazebo_description/woody/gazebo_urdf/woody.gazebo.xacro (robot description, xacro)
@@ -2,246 +2,46 @@
 <robot name="woody"
        xmlns:xacro="http://ros.org/wiki/xacro" >
-<!-- Import Files ######################################################### -->
-  <!-- ==================================================================== -->
-  <xacro:include filename="$(find pandora_robots_description)/urdf/woody/woody.urdf.xacro" />
-  <!-- ==================================================================== -->
-  <xacro:include filename="$(find pandora_gazebo_description)/urdf/woody/sdf_configurations.xacro" />
-  <!-- ==================================================================== -->
-  <xacro:include filename="$(find pandora_gazebo_description)/urdf/woody/physics/robot_physics.gazebo.xacro" />
-  <!-- ==================================================================== -->
-  <xacro:include filename="$(find pandora_gazebo_description)/urdf/woody/physics/wheel_link_physics.gazebo.xacro" />
-  <!-- ==================================================================== -->
-  <xacro:include filename="$(find pandora_gazebo_description)/urdf/woody/physics/side_joint_physics.gazebo.xacro" />
-  <xacro:include filename="$(find pandora_gazebo_description)/urdf/woody/physics/wheel_joint_physics.gazebo.xacro" />
-  <xacro:include filename="$(find pandora_gazebo_description)/urdf/woody/physics/laser_roll_joint_physics.gazebo.xacro" />
-  <xacro:include filename="$(find pandora_gazebo_description)/urdf/woody/physics/laser_pitch_joint_physics.gazebo.xacro" />
-  <xacro:include filename="$(find pandora_gazebo_description)/urdf/woody/physics/kinect_pitch_joint_physics.gazebo.xacro" />
-  <xacro:include filename="$(find pandora_gazebo_description)/urdf/woody/physics/kinect_yaw_joint_physics.gazebo.xacro" />
-  <!-- ==================================================================== -->
-  <xacro:include filename="$(find pandora_gazebo_description)/urdf/woody/sensors/laser_sensor.gazebo.xacro" />
-  <xacro:include filename="$(find pandora_gazebo_description)/urdf/woody/sensors/kinect_sensor.gazebo.xacro" />
-  <xacro:include filename="$(find pandora_gazebo_description)/urdf/woody/sensors/camera_sensor.gazebo.xacro" />
-  <xacro:include filename="$(find pandora_gazebo_description)/urdf/woody/sensors/sonar_sensor.gazebo.xacro" />
-  <xacro:include filename="$(find pandora_gazebo_description)/urdf/woody/sensors/thermal_sensor.gazebo.xacro" />
-  <xacro:include filename="$(find pandora_gazebo_description)/urdf/woody/sensors/co2_sensor.gazebo.xacro" />
-  <xacro:include filename="$(find pandora_gazebo_description)/urdf/woody/sensors/microphone_sensor.gazebo.xacro" />
-  <!-- ==================================================================== -->
-  <xacro:include filename="$(find pandora_gazebo_description)/urdf/woody/transmissions/wheel_transmission.xacro" />
-  <xacro:include filename="$(find pandora_gazebo_description)/urdf/woody/transmissions/laser_sensor_transmission.xacro" />
-  <xacro:include filename="$(find pandora_gazebo_description)/urdf/woody/transmissions/kinect_sensor_transmission.xacro" />
-  <!-- ==================================================================== -->
-  <xacro:include filename="$(find pandora_gazebo_description)/urdf/woody/plugins/pandora_differential_plugin.gazebo.xacro" />
-  <xacro:include filename="$(find pandora_gazebo_description)/urdf/woody/plugins/pandora_p3d_plugin.gazebo.xacro" />
-  <xacro:include filename="$(find pandora_gazebo_description)/urdf/woody/plugins/pandora_imu_stabilizer_plugin.gazebo.xacro" />
-  <xacro:include filename="$(find pandora_gazebo_description)/urdf/woody/plugins/ros_imu_plugin.gazebo.xacro" />
-  <xacro:include filename="$(find pandora_gazebo_description)/urdf/woody/plugins/ros_skid_steer_drive_plugin.gazebo.xacro" />
-  <xacro:include filename="$(find pandora_gazebo_description)/urdf/woody/plugins/ros_control_plugin.gazebo.xacro" />
-  <xacro:include filename="$(find pandora_gazebo_description)/urdf/woody/plugins/pandora_wheel_physics_plugin.gazebo.xacro" />
-  <xacro:include filename="$(find pandora_gazebo_description)/urdf/woody/plugins/pandora_fdir_plugin.gazebo.xacro" />
-  <!-- ==================================================================== -->
-<!-- Load URDF ############################################################ -->
-  <!-- ==================================================================== -->
-  <xacro:if value="$(arg control)" >
-    <xacro:woody_urdf fixed="false" />
+  <!-- Import Files -->
+  <xacro:include filename="$(find pandora_robots_description)/woody/urdf/woody.urdf.xacro" />
+  <xacro:include filename="$(find pandora_gazebo_description)/sensors/*.gazebo.xacro" />
+  <xacro:include filename="$(find pandora_gazebo_description)/plugins/*.gazebo.xacro" />
+  <!-- Load URDF -->
+  <xacro:woody_urdf />
+  <!-- Load gazebo sensors -->
+  <xacro:if value="$(arg enable_laser)" >
+    <xacro:laser_sensor range="4" />
   </xacro:if>
-  <!-- ==================================================================== -->
-  <xacro:unless value="$(arg control)" >
-    <xacro:woody_urdf fixed="true" />
-  </xacro:unless>
-  <!-- ==================================================================== -->
-<!-- Load Physics ######################################################### -->
-  <xacro:robot_physics />
-  <xacro:if value="${enable_gazebo_physics}" >
-    <xacro:if value="${enable_side_joint_physics}" >
-      <xacro:side_joint_physics prefix_y="left" />
-      <xacro:side_joint_physics prefix_y="right" />
-    </xacro:if>
-    <!-- ================================================================ -->
-    <xacro:if value="${enable_wheel_link_physics}" >
-      <xacro:wheel_link_physics prefix_y="left" prefix_x="front" />
-      <xacro:wheel_link_physics prefix_y="left" prefix_x="rear" />
-      <xacro:wheel_link_physics prefix_y="right" prefix_x="front" />
-      <xacro:wheel_link_physics prefix_y="right" prefix_x="rear" />
-    </xacro:if>
-    <!-- ================================================================ -->
-    <xacro:if value="${enable_wheel_joint_physics}" >
-      <xacro:wheel_joint_physics prefix_y="left" prefix_x="front" />
-      <xacro:wheel_joint_physics prefix_y="left" prefix_x="rear" />
-      <xacro:wheel_joint_physics prefix_y="right" prefix_x="front" />
-      <xacro:wheel_joint_physics prefix_y="right" prefix_x="rear" />
-    </xacro:if>
-    <!-- ================================================================ -->
-    <xacro:if value="${enable_sensors}" >
-      <!-- ================================================================ -->
-      <xacro:if value="${enable_laser_sensor}" >
-        <!-- ============================================================== -->
-        <xacro:if value="${enable_laser_roll_joint_physics}" >
-          <xacro:laser_roll_joint_physics />
-        </xacro:if>
-        <!-- ============================================================== -->
-        <xacro:if value="${enable_laser_pitch_joint_physics}" >
-          <xacro:laser_pitch_joint_physics />
-        </xacro:if>
-        <!-- ============================================================== -->
-      </xacro:if>
-      <!-- ================================================================ -->
-      <xacro:if value="${enable_kinect_sensor}" >
-        <!-- ============================================================== -->
-        <xacro:if value="${enable_kinect_pitch_joint_physics}" >
-          <xacro:kinect_pitch_joint_physics />
-        </xacro:if>
-        <!-- ============================================================== -->
-        <xacro:if value="${enable_kinect_yaw_joint_physics}" >
-          <xacro:kinect_yaw_joint_physics />
-        </xacro:if>
-        <!-- ============================================================== -->
-      </xacro:if>
-      <!-- ================================================================ -->
-    </xacro:if>
+  <xacro:if value="$(arg enable_kinect)" >
+    <xacro:kinect_sensor />
   </xacro:if>
-<!-- Load Gazebo Sensors ################################################## -->
-  <xacro:if value="${enable_sensors}" >
-    <xacro:if value="${enable_gazebo_sensors}" >
-      <xacro:if value="${enable_laser_sensor}" >
-        <xacro:if value="${enable_laser_gazebo_sensor}" >
-          <xacro:laser_gazebo_sensor />
-        </xacro:if>
-      </xacro:if>
-      <xacro:if value="${enable_kinect_sensor}" >
-        <xacro:if value="${enable_kinect_gazebo_sensor}" >
-          <xacro:kinect_gazebo_sensor />
-        </xacro:if>
-      </xacro:if>
-      <xacro:if value="${enable_camera_sensors}" >
-        <xacro:if value="${enable_camera_gazebo_sensors}" >
-          <!-- ============================================================ -->
-          <xacro:if value="${enable_left_camera_sensor}" >
-            <xacro:if value="${enable_left_camera_gazebo_sensor}" >
-              <xacro:camera_gazebo_sensor prefix_y="left" />
-            </xacro:if>
-          </xacro:if>
-          <!-- ============================================================ -->
-          <xacro:if value="${enable_right_camera_sensor}" >
-            <xacro:if value="${enable_right_camera_gazebo_sensor}" >
-              <xacro:camera_gazebo_sensor prefix_y="right" />
-            </xacro:if>
-          </xacro:if>
-          <!-- ============================================================ -->
-        </xacro:if>
-      </xacro:if>
-      <xacro:if value="${enable_sonar_sensors}" >
-        <xacro:if value="${enable_sonar_gazebo_sensors}" >
-          <!-- ============================================================ -->
-          <xacro:if value="${enable_left_sonar_sensor}" >
-            <xacro:if value="${enable_left_sonar_gazebo_sensor}" >
-              <xacro:sonar_gazebo_sensor name="left" />
-            </xacro:if>
-          </xacro:if>
-          <!-- ============================================================ -->
-          <xacro:if value="${enable_right_sonar_sensor}" >
-            <xacro:if value="${enable_right_sonar_gazebo_sensor}" >
-              <xacro:sonar_gazebo_sensor name="right" />
-            </xacro:if>
-          </xacro:if>
-          <!-- ============================================================ -->
-        </xacro:if>
-      </xacro:if>
-      <xacro:if value="${enable_co2_sensor}" >
-        <xacro:if value="${enable_co2_gazebo_sensor}" >
-          <xacro:co2_gazebo_sensor />
-        </xacro:if>
-      </xacro:if>
-      <xacro:if value="${enable_thermal_sensor}" >
-        <xacro:if value="${enable_thermal_gazebo_sensor}" >
-          <xacro:if value="${enable_thermal_gazebo_sensor}" >
-            <xacro:thermal_gazebo_sensor prefix_y="middle" />
-          </xacro:if>
-        </xacro:if>
-      </xacro:if>
-      <xacro:if value="${enable_microphone_sensor}" >
-        <xacro:if value="${enable_microphone_gazebo_sensor}" >
-          <xacro:microphone_gazebo_sensor />
-        </xacro:if>
-      </xacro:if>
-    </xacro:if>
+  <xacro:if value="$(arg enable_webcam)" >
+    <xacro:thermal_sensor />
   </xacro:if>
-<!-- Load Transmissions ################################################### -->
-  <xacro:if value="$(arg control)" >
-    <xacro:wheel_transmission prefix_y="left" prefix_x="front" />
-    <xacro:wheel_transmission prefix_y="left" prefix_x="rear" />
-    <xacro:wheel_transmission prefix_y="right" prefix_x="front" />
-    <xacro:wheel_transmission prefix_y="right" prefix_x="rear" />
-    <xacro:if value="${enable_sensors}" >
-      <!-- ================================================================ -->
-      <xacro:if value="${enable_laser_sensor}" >
-        <xacro:laser_sensor_transmission rotation="roll" />
-        <xacro:laser_sensor_transmission rotation="pitch" />
-      </xacro:if>
-      <!-- ================================================================ -->
-      <xacro:if value="${enable_kinect_sensor}" >
-        <xacro:kinect_sensor_transmission rotation="pitch" />
-        <xacro:kinect_sensor_transmission rotation="yaw" />
-      </xacro:if>
-      <!-- ================================================================ -->
-    </xacro:if>
+  <xacro:if value="$(arg enable_sonar)" >
+    <xacro:webcam_sensor prefix_y="left" />
+    <xacro:webcam_sensor prefix_y="right" />
   </xacro:if>
-<!-- Load Plugins ######################################################### -->
-  <xacro:if value="${enable_plugins}" >
-    <xacro:if value="${enable_pandora_differential_plugin}" >
-      <xacro:if value="$(arg control)" >
-        <!-- ============================================================== -->
-        <xacro:if value="$(arg interface)" >
-          <xacro:pandora_differential_plugin publish_joint_states="false" />
-        </xacro:if>
-        <!-- ============================================================== -->
-        <xacro:unless value="$(arg interface)" >
-          <xacro:pandora_differential_plugin publish_joint_states="true" />
-        </xacro:unless>
-        <!-- ============================================================== -->
-      </xacro:if>
-      <xacro:unless value="$(arg control)" >
-        <xacro:pandora_differential_plugin publish_joint_states="true" />
-      </xacro:unless>
-    </xacro:if>
-    <xacro:if value="${enable_pandora_p3d_plugin}" >
-      <xacro:pandora_p3d_plugin />
-    </xacro:if>
-    <xacro:unless value="$(arg control)" >
-      <xacro:if value="${enable_sensors}" >
-        <xacro:if value="${enable_laser_sensor}" >
-          <xacro:if value="${enable_pandora_imu_stabilizer_plugin}" >
-            <!-- <xacro:pandora_imu_stabilizer_plugin /> --> <!-- FIXME -->
-          </xacro:if>
-        </xacro:if>
-      </xacro:if>
-    </xacro:unless>
-    <xacro:if value="$(arg control)" >
-      <xacro:unless value="$(arg interface)" >
-        <xacro:if value="${enable_ros_imu_plugin}" >
-          <xacro:ros_imu_plugin />
-        </xacro:if>
-      </xacro:unless>
-    </xacro:if>
-    <xacro:unless value="$(arg control)" >
-      <xacro:if value="${enable_ros_skid_steer_drive_plugin}" >
-        <xacro:ros_skid_steer_drive_plugin />
-      </xacro:if>
-    </xacro:unless>
+  <xacro:if value="$(arg enable_thermal)" >
+    <xacro:sonar_sensor name="left" />
+    <xacro:sonar_sensor name="right" />
   </xacro:if>
-<!-- Load Ros Control ##################################################### -->
-  <xacro:if value="$(arg control)" >
-    <xacro:if value="$(arg interface)" >
-      <xacro:gazebo_ros_control_plugin namespace="/"
-                                       hardware_interface="pandora_gazebo_interface/WoodyGazeboInterface" />
-    </xacro:if>
-    <xacro:unless value="$(arg interface)" >
-      <xacro:gazebo_ros_control_plugin namespace="/"
-                                       hardware_interface="gazebo_ros_control/DefaultRobotHWSim" />
-    </xacro:unless>
+  <xacro:if value="$(arg enable_temperature)" >
+    <xacro:co2_sensor />
   </xacro:if>
-<!-- Enable tuning ######################################################## -->
-  <xacro:if value="$(arg tune)">
+  <xacro:if value="$(arg enable_co2)" >
+    <xacro:temperature_sensor prefix_y="middle" />
+    <xacro:temperature_sensor prefix_y="left" />
+    <xacro:temperature_sensor prefix_y="right" />
+  </xacro:if>
+  <xacro:if value="$(arg enable_microphone)" >
+    <xacro:microphone_sensor />
+  </xacro:if>
+  <!-- Load Plugins -->
+  <xacro:pandora_differential_plugin />
+  <xacro:pandora_p3d_plugin />
+  <xacro:gazebo_ros_control_plugin interface="pandora_gazebo_interface/WoodyGazeboInterface" />
+  <xacro:if value="$(arg tune)" >
     <xacro:pandora_wheel_physics_plugin/>
+    <!--<xacro:pandora_fdir_plugin />-->
   </xacro:if>
-<!--<xacro:pandora_fdir_plugin/>-->
 </robot>
