Commit message: Remove ros_control arg from world launchers

File: pandora_gazebo_description/woody/gazebo_urdf/sdf_configurations.xacro (robot description, xacro)
@@ -1,4 +1,6 @@
 <?xml version="1.0"?>
 <robot xmlns:xacro="http://ros.org/wiki/xacro" >
+  <!-- Sensor properties -->
+  <xacro:property name="laser_range" value="4" />
   <!-- Enable gazebo sensors -->
   <xacro:property name="enable_laser" value="true" />

File: pandora_gazebo_description/woody/gazebo_urdf/woody.gazebo.xacro (robot description, xacro)
@@ -10,5 +10,5 @@
   <!-- Load gazebo sensors -->
   <xacro:if value="$(arg enable_laser)" >
-    <xacro:laser_sensor range="4" />
+    <xacro:laser_sensor range="$(arg laser_range)" />
   </xacro:if>
   <xacro:if value="$(arg enable_kinect)" >
@@ -38,7 +38,7 @@
   </xacro:if>
   <!-- Load Plugins -->
+  <xacro:gazebo_ros_control_plugin interface="pandora_gazebo_interface/WoodyGazeboInterface" />
   <xacro:pandora_differential_plugin />
   <xacro:pandora_p3d_plugin />
-  <xacro:gazebo_ros_control_plugin interface="pandora_gazebo_interface/WoodyGazeboInterface" />
   <xacro:if value="$(arg tune)" >
     <xacro:pandora_wheel_physics_plugin/>
