Commit message: Finish woody_gazebo_description refactoring

File: pandora_gazebo_description/sdf_elements/plugins/ros_control_plugin.gazebo.xacro (robot description, xacro)
@@ -1,5 +1,5 @@
 <?xml version="1.0"?>
 <robot xmlns:xacro="http://ros.org/wiki/xacro" >
-  <xacro:macro name="gazebo_ros_control_plugin" params="interface" >
+  <xacro:macro name="gazebo_ros_control" params="interface" >
     <gazebo>
       <plugin name="GazeboRosControl" filename="libgazebo_ros_control.so" >
