Commit message: Remove redundant temperature gazebo sensors

File: pandora_gazebo_description/woody/urdf_gazebo/sdf_configurations.xacro (robot description, xacro)
@@ -6,9 +6,9 @@
   <xacro:property name="enable_laser" value="true" />
   <xacro:property name="enable_kinect" value="true" />
+  <xacro:property name="enable_thermal" value="false" />
   <xacro:property name="enable_webcam" value="true" />
   <xacro:property name="enable_sonar" value="true" />
-  <xacro:property name="enable_thermal" value="false" />
+  <xacro:property name="enable_co2" value="true" />
   <xacro:property name="enable_temperature" value="false" />
-  <xacro:property name="enable_co2" value="true" />
   <xacro:property name="enable_microphone" value="false" />
   <!-- Wheel physics -->

File: pandora_gazebo_description/woody/urdf_gazebo/woody.gazebo.xacro (robot description, xacro)
@@ -17,22 +17,20 @@
     <xacro:kinect_sensor />
   </xacro:if>
-  <xacro:if value="${enable_webcam}" >
+  <xacro:if value="${enable_thermal}" >
     <xacro:thermal_sensor />
   </xacro:if>
-  <xacro:if value="${enable_sonar}" >
+  <xacro:if value="${enable_webcam}" >
     <xacro:webcam_sensor prefix_y="left" />
     <xacro:webcam_sensor prefix_y="right" />
   </xacro:if>
-  <xacro:if value="${enable_thermal}" >
+  <xacro:if value="${enable_sonar}" >
     <xacro:sonar_sensor name="left" />
     <xacro:sonar_sensor name="right" />
   </xacro:if>
-  <xacro:if value="${enable_temperature}" >
+  <xacro:if value="${enable_co2}" >
     <xacro:co2_sensor />
   </xacro:if>
-  <xacro:if value="${enable_co2}" >
+  <xacro:if value="${enable_temperature}" >
     <xacro:temperature_sensor prefix_y="middle" />
-    <xacro:temperature_sensor prefix_y="left" />
-    <xacro:temperature_sensor prefix_y="right" />
   </xacro:if>
   <xacro:if value="${enable_microphone}" >
