Commit message: Add thermal sensor gazebo reference

File: pandora_gazebo_description/sdf_elements/sensors/temperature_sensor.gazebo.xacro (robot description, xacro)
@@ -1,22 +1,22 @@
 <?xml version="1.0"?>
 <robot xmlns:xacro="http://ros.org/wiki/xacro" >
-  <xacro:macro name="thermal_sensor" >
-    <gazebo reference="flir_frame" >
-      <sensor name="thermal" type="camera" >
+  <xacro:macro name="temperature_sensor" params="prefix_y" >
+    <gazebo reference="${prefix_y}_thermal_frame" >
+      <sensor name="${prefix_y}_thermal" type="camera" >
         <camera>
           <horizontal_fov>0.8</horizontal_fov>
           <image>
-            <width>80</width>
-            <height>60</height>
+            <width>8</width>
+            <height>8</height>
           </image>
           <clip>
-            <near>0.1</near>
-            <far>3.0</far>
+            <near>0.05</near>
+            <far>1.5</far>
           </clip>
         </camera>
         <plugin name="thermal2ros" filename="libpandora_gazebo_plugins_pandora_thermal_plugin.so" >
           <robotNamespace>gazebo_sensors</robotNamespace>
-          <frameName>flir_optical_frame</frameName>
-          <topicName>flir</topicName>
+          <frameName>${prefix_y}_thermal_optical_frame</frameName>
+          <topicName>thermal</topicName>
         </plugin>
         <always_on>1</always_on>
