Commit message: Complete gears_gazebo_description refactoring

File: pandora_gazebo_description/gears/urdf_gazebo/gears.gazebo.xacro (robot description, xacro)
@@ -2,289 +2,46 @@
 <robot name="gears"
        xmlns:xacro="http://ros.org/wiki/xacro" >
-<!-- Import Files ######################################################### -->
-  <!-- ==================================================================== -->
-  <xacro:include filename="$(find pandora_robots_description)/urdf/gears/gears.urdf.xacro" />
-  <!-- ==================================================================== -->
-  <xacro:include filename="$(find pandora_gazebo_description)/urdf/gears/sdf_configurations.xacro" />
-  <!-- ==================================================================== -->
-  <xacro:include filename="$(find pandora_gazebo_description)/urdf/gears/physics/robot_physics.gazebo.xacro" />
-  <!-- ==================================================================== -->
-  <xacro:include filename="$(find pandora_gazebo_description)/urdf/gears/physics/wheel_link_physics.gazebo.xacro" />
-  <!-- ==================================================================== -->
-  <xacro:include filename="$(find pandora_gazebo_description)/urdf/gears/physics/side_joint_physics.gazebo.xacro" />
-  <xacro:include filename="$(find pandora_gazebo_description)/urdf/gears/physics/wheel_joint_physics.gazebo.xacro" />
-  <xacro:include filename="$(find pandora_gazebo_description)/urdf/gears/physics/linear_elevator_joint_physics.gazebo.xacro" />
-  <xacro:include filename="$(find pandora_gazebo_description)/urdf/gears/physics/linear_head_pitch_joint_physics.gazebo.xacro" />
-  <xacro:include filename="$(find pandora_gazebo_description)/urdf/gears/physics/linear_head_yaw_joint_physics.gazebo.xacro" />
-  <xacro:include filename="$(find pandora_gazebo_description)/urdf/gears/physics/laser_roll_joint_physics.gazebo.xacro" />
-  <xacro:include filename="$(find pandora_gazebo_description)/urdf/gears/physics/laser_pitch_joint_physics.gazebo.xacro" />
-  <xacro:include filename="$(find pandora_gazebo_description)/urdf/gears/physics/kinect_pitch_joint_physics.gazebo.xacro" />
-  <xacro:include filename="$(find pandora_gazebo_description)/urdf/gears/physics/kinect_yaw_joint_physics.gazebo.xacro" />
-  <!-- ==================================================================== -->
-  <xacro:include filename="$(find pandora_gazebo_description)/urdf/gears/sensors/laser_sensor.gazebo.xacro" />
-  <xacro:include filename="$(find pandora_gazebo_description)/urdf/gears/sensors/kinect_sensor.gazebo.xacro" />
-  <xacro:include filename="$(find pandora_gazebo_description)/urdf/gears/sensors/camera_sensor.gazebo.xacro" />
-  <xacro:include filename="$(find pandora_gazebo_description)/urdf/gears/sensors/sonar_sensor.gazebo.xacro" />
-  <xacro:include filename="$(find pandora_gazebo_description)/urdf/gears/sensors/thermal_sensor.gazebo.xacro" />
-  <xacro:include filename="$(find pandora_gazebo_description)/urdf/gears/sensors/co2_sensor.gazebo.xacro" />
-  <xacro:include filename="$(find pandora_gazebo_description)/urdf/gears/sensors/microphone_sensor.gazebo.xacro" />
-  <!-- ==================================================================== -->
-  <xacro:include filename="$(find pandora_gazebo_description)/urdf/gears/transmissions/wheel_transmission.xacro" />
-  <xacro:include filename="$(find pandora_gazebo_description)/urdf/gears/transmissions/linear_elevator_transmission.xacro" />
-  <xacro:include filename="$(find pandora_gazebo_description)/urdf/gears/transmissions/linear_head_transmission.xacro" />
-  <xacro:include filename="$(find pandora_gazebo_description)/urdf/gears/transmissions/laser_sensor_transmission.xacro" />
-  <xacro:include filename="$(find pandora_gazebo_description)/urdf/gears/transmissions/kinect_sensor_transmission.xacro" />
-  <!-- ==================================================================== -->
-  <xacro:include filename="$(find pandora_gazebo_description)/urdf/gears/plugins/pandora_differential_plugin.gazebo.xacro" />
-  <xacro:include filename="$(find pandora_gazebo_description)/urdf/gears/plugins/pandora_p3d_plugin.gazebo.xacro" />
-  <xacro:include filename="$(find pandora_gazebo_description)/urdf/gears/plugins/pandora_imu_stabilizer_plugin.gazebo.xacro" />
-  <xacro:include filename="$(find pandora_gazebo_description)/urdf/gears/plugins/ros_imu_plugin.gazebo.xacro" />
-  <xacro:include filename="$(find pandora_gazebo_description)/urdf/gears/plugins/ros_skid_steer_drive_plugin.gazebo.xacro" />
-  <xacro:include filename="$(find pandora_gazebo_description)/urdf/gears/plugins/ros_control_plugin.gazebo.xacro" />
-  <xacro:include filename="$(find pandora_gazebo_description)/urdf/gears/plugins/pandora_wheel_physics_plugin.gazebo.xacro" />
-  <xacro:include filename="$(find pandora_gazebo_description)/urdf/gears/plugins/pandora_fdir_plugin.gazebo.xacro" />
-  <!-- ==================================================================== -->
-<!-- Load URDF ############################################################ -->
-  <!-- ==================================================================== -->
-  <xacro:if value="$(arg control)" >
-    <xacro:gears_urdf fixed="false" />
+  <!-- Import Files -->
+  <xacro:include filename="$(find pandora_robots_description)/gears/urdf/gears.urdf.xacro" />
+  <xacro:include filename="$(find pandora_gazebo_description)/gears/urdf_gazebo/sdf_configurations.xacro" />
+  <xacro:include filename="$(find pandora_gazebo_description)/gears/urdf_gazebo/physics.gazebo.xacro" />
+  <xacro:include filename="$(find pandora_gazebo_description)/sdf_elements/sensors/*.gazebo.xacro" />
+  <xacro:include filename="$(find pandora_gazebo_description)/sdf_elements/plugins/*.gazebo.xacro" />
+  <!-- Load URDF -->
+  <xacro:gears_urdf />
+  <!-- Load gazebo sensors -->
+  <xacro:if value="${enable_laser}" >
+    <xacro:laser_sensor range="${laser_range}" />
   </xacro:if>
-  <!-- ==================================================================== -->
-  <xacro:unless value="$(arg control)" >
-    <xacro:gears_urdf fixed="true" />
-  </xacro:unless>
-  <!-- ==================================================================== -->
-<!-- Load Physics ######################################################### -->
-  <xacro:robot_physics />
-  <xacro:if value="${enable_gazebo_physics}" >
-    <xacro:if value="${enable_side_joint_physics}" >
-      <xacro:side_joint_physics prefix_y="left" />
-      <xacro:side_joint_physics prefix_y="right" />
-    </xacro:if>
-    <!-- ================================================================ -->
-    <xacro:if value="${enable_wheel_link_physics}" >
-      <xacro:wheel_link_physics prefix_y="left" prefix_x="front" />
-      <xacro:wheel_link_physics prefix_y="left" prefix_x="rear" />
-      <xacro:wheel_link_physics prefix_y="right" prefix_x="front" />
-      <xacro:wheel_link_physics prefix_y="right" prefix_x="rear" />
-    </xacro:if>
-    <!-- ================================================================ -->
-    <xacro:if value="${enable_wheel_joint_physics}" >
-      <xacro:wheel_joint_physics prefix_y="left" prefix_x="front" />
-      <xacro:wheel_joint_physics prefix_y="left" prefix_x="rear" />
-      <xacro:wheel_joint_physics prefix_y="right" prefix_x="front" />
-      <xacro:wheel_joint_physics prefix_y="right" prefix_x="rear" />
-    </xacro:if>
-    <!-- ================================================================ -->
-    <!-- ================================================================ -->
-    <xacro:if value="${enable_linear_elevator_joint_physics}" >
-      <xacro:linear_elevator_joint_physics />
-    </xacro:if>
-    <!-- ================================================================ -->
-    <xacro:if value="${enable_linear_head_yaw_joint_physics}" >
-      <xacro:linear_head_yaw_joint_physics />
-    </xacro:if>
-    <!-- ================================================================ -->
-    <xacro:if value="${enable_linear_head_pitch_joint_physics}" >
-      <xacro:linear_head_pitch_joint_physics />
-    </xacro:if>
-    <!-- ================================================================ -->
-    <xacro:if value="${enable_sensors}" >
-      <!-- ================================================================ -->
-      <xacro:if value="${enable_laser_sensor}" >
-        <!-- ============================================================== -->
-        <xacro:if value="${enable_laser_roll_joint_physics}" >
-          <xacro:laser_roll_joint_physics />
-        </xacro:if>
-        <!-- ============================================================== -->
-        <xacro:if value="${enable_laser_pitch_joint_physics}" >
-          <xacro:laser_pitch_joint_physics />
-        </xacro:if>
-        <!-- ============================================================== -->
-      </xacro:if>
-      <!-- ================================================================ -->
-      <xacro:if value="${enable_kinect_sensor}" >
-        <!-- ============================================================== -->
-        <xacro:if value="${enable_kinect_pitch_joint_physics}" >
-          <xacro:kinect_pitch_joint_physics />
-        </xacro:if>
-        <!-- ============================================================== -->
-        <xacro:if value="${enable_kinect_yaw_joint_physics}" >
-          <xacro:kinect_yaw_joint_physics />
-        </xacro:if>
-        <!-- ============================================================== -->
-      </xacro:if>
-      <!-- ================================================================ -->
-    </xacro:if>
+  <xacro:if value="${enable_kinect}" >
+    <xacro:kinect_sensor />
   </xacro:if>
-<!-- Load Gazebo Sensors ################################################## -->
-  <xacro:if value="${enable_sensors}" >
-    <xacro:if value="${enable_gazebo_sensors}" >
-      <xacro:if value="${enable_laser_sensor}" >
-        <xacro:if value="${enable_laser_gazebo_sensor}" >
-          <xacro:laser_gazebo_sensor />
-        </xacro:if>
-      </xacro:if>
-      <xacro:if value="${enable_kinect_sensor}" >
-        <xacro:if value="${enable_kinect_gazebo_sensor}" >
-          <xacro:kinect_gazebo_sensor />
-        </xacro:if>
-      </xacro:if>
-      <xacro:if value="${enable_camera_sensors}" >
-        <xacro:if value="${enable_camera_gazebo_sensors}" >
-          <!-- ============================================================ -->
-          <xacro:if value="${enable_left_camera_sensor}" >
-            <xacro:if value="${enable_left_camera_gazebo_sensor}" >
-              <xacro:camera_gazebo_sensor prefix_y="left" />
-            </xacro:if>
-          </xacro:if>
-          <!-- ============================================================ -->
-          <xacro:if value="${enable_right_camera_sensor}" >
-            <xacro:if value="${enable_right_camera_gazebo_sensor}" >
-              <xacro:camera_gazebo_sensor prefix_y="right" />
-            </xacro:if>
-          </xacro:if>
-          <!-- ============================================================ -->
-        </xacro:if>
-      </xacro:if>
-      <xacro:if value="${enable_sonar_sensors}" >
-        <xacro:if value="${enable_sonar_gazebo_sensors}" >
-          <!-- ============================================================ -->
-          <xacro:if value="${enable_linear_sonar_sensor}" >
-            <xacro:if value="${enable_linear_sonar_gazebo_sensor}" >
-              <xacro:sonar_gazebo_sensor name="linear" />
-            </xacro:if>
-          </xacro:if>
-          <!-- ============================================================ -->
-          <xacro:if value="${enable_left_sonar_sensor}" >
-            <xacro:if value="${enable_left_sonar_gazebo_sensor}" >
-                  <xacro:sonar_gazebo_sensor name="left" />
-            </xacro:if>
-          </xacro:if>
-          <!-- ============================================================ -->
-          <xacro:if value="${enable_right_sonar_sensor}" >
-            <xacro:if value="${enable_right_sonar_gazebo_sensor}" >
-                  <xacro:sonar_gazebo_sensor name="right" />
-            </xacro:if>
-          </xacro:if>
-          <!-- ============================================================ -->
-        </xacro:if>
-      </xacro:if>
-      <xacro:if value="${enable_co2_sensor}" >
-        <xacro:if value="${enable_co2_gazebo_sensor}" >
-                <xacro:co2_gazebo_sensor />
-        </xacro:if>
-      </xacro:if>
-      <xacro:if value="${enable_thermal_sensors}" >
-        <xacro:if value="${enable_thermal_gazebo_sensors}" >
-          <!-- ============================================================ -->
-          <xacro:if value="${enable_middle_thermal_sensor}" >
-            <xacro:if value="${enable_middle_thermal_gazebo_sensor}" >
-                    <xacro:thermal_gazebo_sensor prefix_y="middle" />
-            </xacro:if>
-          </xacro:if>
-          <!-- ============================================================ -->
-          <xacro:if value="${enable_left_thermal_sensor}" >
-            <xacro:if value="${enable_left_thermal_gazebo_sensor}" >
-                    <xacro:thermal_gazebo_sensor prefix_y="left" />
-            </xacro:if>
-          </xacro:if>
-          <!-- ============================================================ -->
-          <xacro:if value="${enable_right_thermal_sensor}" >
-            <xacro:if value="${enable_right_thermal_gazebo_sensor}" >
-                    <xacro:thermal_gazebo_sensor prefix_y="right" />
-            </xacro:if>
-          </xacro:if>
-          <!-- ============================================================ -->
-        </xacro:if>
-      </xacro:if>
-      <xacro:if value="${enable_microphone_sensor}" >
-        <xacro:if value="${enable_microphone_gazebo_sensor}" >
-                <xacro:microphone_gazebo_sensor />
-        </xacro:if>
-      </xacro:if>
-    </xacro:if>
+  <xacro:if value="${enable_webcam}" >
+    <xacro:webcam_sensor prefix_y="left" />
+    <xacro:webcam_sensor prefix_y="right" />
   </xacro:if>
-<!-- Load Transmissions ################################################### -->
-  <xacro:if value="$(arg control)" >
-    <xacro:wheel_transmission prefix_y="left" prefix_x="front" />
-    <xacro:wheel_transmission prefix_y="left" prefix_x="rear" />
-    <xacro:wheel_transmission prefix_y="right" prefix_x="front" />
-    <xacro:wheel_transmission prefix_y="right" prefix_x="rear" />
-    <xacro:linear_elevator_transmission />
-    <xacro:linear_head_transmission rotation="pitch" />
-    <xacro:linear_head_transmission rotation="yaw" />
-    <xacro:if value="${enable_sensors}" >
-      <!-- ================================================================ -->
-      <xacro:if value="${enable_laser_sensor}" >
-        <xacro:laser_sensor_transmission rotation="roll" />
-        <xacro:laser_sensor_transmission rotation="pitch" />
-      </xacro:if>
-      <!-- ================================================================ -->
-      <xacro:if value="${enable_kinect_sensor}" >
-        <xacro:kinect_sensor_transmission rotation="pitch" />
-        <xacro:kinect_sensor_transmission rotation="yaw" />
-      </xacro:if>
-      <!-- ================================================================ -->
-    </xacro:if>
+  <xacro:if value="${enable_sonar}" >
+    <xacro:sonar_sensor name="linear" />
+    <xacro:sonar_sensor name="left" />
+    <xacro:sonar_sensor name="right" />
   </xacro:if>
-<!-- Load Plugins ######################################################### -->
-  <xacro:if value="${enable_plugins}" >
-    <xacro:if value="${enable_pandora_differential_plugin}" >
-      <xacro:if value="$(arg control)" >
-        <!-- ============================================================== -->
-        <xacro:if value="$(arg interface)" >
-          <xacro:pandora_differential_plugin publish_joint_states="false" />
-        </xacro:if>
-        <!-- ============================================================== -->
-        <xacro:unless value="$(arg interface)" >
-          <xacro:pandora_differential_plugin publish_joint_states="true" />
-        </xacro:unless>
-        <!-- ============================================================== -->
-      </xacro:if>
-      <xacro:unless value="$(arg control)" >
-        <xacro:pandora_differential_plugin publish_joint_states="true" />
-      </xacro:unless>
-    </xacro:if>
-    <xacro:if value="${enable_pandora_p3d_plugin}" >
-      <xacro:pandora_p3d_plugin />
-    </xacro:if>
-    <xacro:unless value="$(arg control)" >
-      <xacro:if value="${enable_sensors}" >
-        <xacro:if value="${enable_laser_sensor}" >
-          <xacro:if value="${enable_pandora_imu_stabilizer_plugin}" >
-            <!-- <xacro:pandora_imu_stabilizer_plugin /> --> <!-- FIXME -->
-          </xacro:if>
-        </xacro:if>
-      </xacro:if>
-    </xacro:unless>
-    <xacro:if value="$(arg control)" >
-      <xacro:unless value="$(arg interface)" >
-        <xacro:if value="${enable_ros_imu_plugin}" >
-          <xacro:ros_imu_plugin />
-        </xacro:if>
-      </xacro:unless>
-    </xacro:if>
-    <xacro:unless value="$(arg control)" >
-      <xacro:if value="${enable_ros_skid_steer_drive_plugin}" >
-        <xacro:ros_skid_steer_drive_plugin />
-      </xacro:if>
-    </xacro:unless>
+  <xacro:if value="${enable_co2}" >
+    <xacro:co2_sensor />
   </xacro:if>
-<!-- Load Ros Control ##################################################### -->
-  <xacro:if value="$(arg control)" >
-    <xacro:if value="$(arg interface)" >
-      <xacro:gazebo_ros_control_plugin namespace="/"
-                                       hardware_interface="pandora_gazebo_interface/GearsGazeboInterface" />
-    </xacro:if>
-    <xacro:unless value="$(arg interface)" >
-      <xacro:gazebo_ros_control_plugin namespace="/"
-                                       hardware_interface="gazebo_ros_control/DefaultRobotHWSim" />
-    </xacro:unless>
+  <xacro:if value="${enable_temperature}" >
+    <xacro:temperature_sensor prefix_y="middle" />
+    <xacro:temperature_sensor prefix_y="left" />
+    <xacro:temperature_sensor prefix_y="right" />
   </xacro:if>
-<!-- Enable tuning ######################################################## -->
-  <xacro:if value="$(arg tune)">
-    <xacro:pandora_wheel_physics_plugin/>
+  <xacro:if value="${enable_microphone}" >
+    <xacro:microphone_sensor />
   </xacro:if>
-<!--<xacro:pandora_fdir_plugin/>-->
+  <!-- Load Plugins -->
+  <xacro:gazebo_ros_control interface="pandora_gazebo_interface/GearsGazeboInterface" />
+  <xacro:pandora_differential />
+  <xacro:pandora_p3d />
+  <xacro:if value="$(arg tune)" >
+    <xacro:pandora_wheel_physics />
+    <!--<xacro:pandora_fdir />-->
+  </xacro:if>
 </robot>
