Commit message: Complete gears_gazebo_description refactoring

File: pandora_gazebo_description/gears/urdf_gazebo/sdf_configurations.xacro (robot description, xacro)
@@ -1,84 +1,20 @@
 <?xml version="1.0"?>
 <robot xmlns:xacro="http://ros.org/wiki/xacro" >
-<!-- Robot NameSpace ###################################################### -->
-  <!-- ==================================================================== -->
-  <xacro:property name="robot_namespace" value="" />
-  <!-- ==================================================================== -->
-<!-- Elements' Status ##################################################### -->
-  <!-- Robot ============================================================== -->
-  <xacro:property name="static_robot" value="false" />
-  <!-- ==================================================================== -->
-  <!-- Sensors ============================================================ -->
-  <xacro:property name="enable_gazebo_sensors" value="true" />
-    <!-- ================================================================== -->
-    <xacro:property name="enable_laser_gazebo_sensor" value="true" />
-    <!-- ================================================================== -->
-    <xacro:property name="enable_kinect_gazebo_sensor" value="true" />
-    <!-- ================================================================== -->
-    <xacro:property name="enable_camera_gazebo_sensors" value="true" />
-      <xacro:property name="enable_left_camera_gazebo_sensor" value="true" />
-      <xacro:property name="enable_right_camera_gazebo_sensor" value="true" />
-    <!-- ================================================================== -->
-    <xacro:property name="enable_sonar_gazebo_sensors" value="true" />
-      <xacro:property name="enable_linear_sonar_gazebo_sensor" value="true" />
-      <xacro:property name="enable_left_sonar_gazebo_sensor" value="true" />
-      <xacro:property name="enable_right_sonar_gazebo_sensor" value="true" />
-    <!-- ================================================================== -->
-    <xacro:property name="enable_thermal_gazebo_sensors" value="true" />
-      <xacro:property name="enable_middle_thermal_gazebo_sensor" value="true" />
-      <xacro:property name="enable_left_thermal_gazebo_sensor" value="true" />
-      <xacro:property name="enable_right_thermal_gazebo_sensor" value="true" />
-    <!-- ================================================================== -->
-    <xacro:property name="enable_co2_gazebo_sensor" value="true" />
-    <!-- ================================================================== -->
-    <xacro:property name="enable_microphone_gazebo_sensor" value="true" />
-  <!-- ==================================================================== -->
-  <!-- Physics ============================================================ -->
-  <xacro:property name="enable_gazebo_physics" value="true" />
-    <!-- Links ============================================================ -->
-    <xacro:property name="enable_wheel_link_physics" value="true" />
-    <!-- ================================================================== -->
-    <!-- Joints =========================================================== -->
-    <xacro:property name="enable_side_joint_physics" value="false" />
-    <!-- ================================================================== -->
-    <xacro:property name="enable_wheel_joint_physics" value="false" />
-    <!-- ================================================================== -->
-    <xacro:property name="enable_linear_elevator_joint_physics" value="true" />
-    <!-- ================================================================== -->
-    <xacro:property name="enable_linear_head_yaw_joint_physics" value="false" />
-    <xacro:property name="enable_linear_head_pitch_joint_physics" value="false" />
-    <!-- ================================================================== -->
-    <xacro:property name="enable_laser_roll_joint_physics" value="false" />
-    <xacro:property name="enable_laser_pitch_joint_physics" value="false" />
-    <!-- ================================================================== -->
-    <xacro:property name="enable_kinect_pitch_joint_physics" value="false" />
-    <xacro:property name="enable_kinect_yaw_joint_physics" value="false" />
-  <!-- ==================================================================== -->
-  <!-- Plugins ============================================================ -->
-  <xacro:property name="enable_plugins" value="true" />
-    <!-- ================================================================== -->
-    <xacro:property name="enable_pandora_differential_plugin" value="true" />
-    <!-- ================================================================== -->
-    <xacro:property name="enable_pandora_p3d_plugin" value="true" />
-    <!-- ================================================================== -->
-    <xacro:property name="enable_pandora_imu_stabilizer_plugin" value="true" />
-    <!-- ================================================================== -->
-    <xacro:property name="enable_ros_imu_plugin" value="true" />
-    <!-- ================================================================== -->
-    <xacro:property name="enable_ros_skid_steer_drive_plugin" value="true" />
-  <!-- ==================================================================== -->
-<!-- Joint Physics ######################################################## -->
-  <!-- Wheels ============================================================= -->
+  <!-- Sensor properties -->
+  <xacro:property name="laser_range" value="4" />
+  <!-- Enable gazebo sensors -->
+  <xacro:property name="enable_laser" value="true" />
+  <xacro:property name="enable_kinect" value="true" />
+  <xacro:property name="enable_webcam" value="true" />
+  <xacro:property name="enable_sonar" value="true" />
+  <xacro:property name="enable_co2" value="true" />
+  <xacro:property name="enable_temperature" value="true" />
+  <xacro:property name="enable_microphone" value="false" />
+  <!-- Wheel physics -->
   <xacro:property name="wheel_mu_1" value="0.85" />
   <xacro:property name="wheel_mu_2" value="0.85" />
-  <xacro:property name="wheel_k_p" value="10000000.0" />
+  <xacro:property name="wheel_k_p" value="1000000.0" />
   <xacro:property name="wheel_k_d" value="1.0" />
-  <xacro:property name="wheel_min_depth" value="0.0001" />
-  <xacro:property name="wheel_max_contacts" value="1" />
-  <!-- ==================================================================== -->
-<!-- Plugin Parameters #################################################### -->
-  <!-- Skid Steer Drive =================================================== -->
-  <xacro:property name="wheel_joint_max_torque" value="5" /> <!-- FIXME -->
-  <!-- ==================================================================== -->
-<!-- ###################################################################### -->
+  <xacro:property name="wheel_min_depth" value="0.001" />
+  <xacro:property name="wheel_max_contacts" value="10" />
 </robot>
