Commit message: Disable unused sensors

File: pandora_gazebo_description/gio/urdf_gazebo/sdf_configurations.xacro (robot description, xacro)
@@ -2,5 +2,5 @@
 <robot xmlns:xacro="http://ros.org/wiki/xacro" >
   <!-- Sensor properties -->
-  <xacro:property name="laser_range" value="4" />
+  <xacro:property name="laser_range" value="20" />
   <!-- Enable gazebo sensors -->
   <xacro:property name="enable_laser" value="true" />
@@ -10,5 +10,5 @@
   <xacro:property name="enable_thermal" value="false" />
   <xacro:property name="enable_sonar" value="true" />
-  <xacro:property name="enable_co2" value="true" />
+  <xacro:property name="enable_co2" value="false" />
   <xacro:property name="enable_microphone" value="false" />
   <!-- Wheel physics -->
