Commit message: Add differential joint in sdf [ci skip]

File: pandora_gazebo_description/gio/urdf_gazebo/gio.gazebo.xacro (robot description, xacro)
@@ -8,6 +8,4 @@
   <xacro:include filename="$(find pandora_gazebo_description)/sdf_elements/sensors/*.gazebo.xacro" />
   <xacro:include filename="$(find pandora_gazebo_description)/sdf_elements/plugins/*.gazebo.xacro" />
-  <!-- Load URDF -->
-  <xacro:gio_urdf />
   <!-- Load gazebo sensors -->
   <xacro:if value="${enable_laser}" >
@@ -39,5 +37,4 @@
   <!-- Load Plugins -->
   <xacro:gazebo_ros_control interface="pandora_gazebo_interface/GioGazeboInterface" />
-  <xacro:pandora_differential />
   <xacro:pandora_p3d />
   <xacro:if value="$(arg tune)" >

File: pandora_gazebo_description/gio/urdf_gazebo/references.gazebo.xacro (robot description, xacro)
@@ -1,4 +1,42 @@
 <?xml version="1.0" ?>
 <robot xmlns:xacro="http://ros.org/wiki/xacro" >
+  <gazebo>
+    <joint name="differential_left_pin_parallel_joint"
+           type="revolute" >
+      <parent>differential_left_pin_link</parent>
+      <child>left_side_link</child>
+      <pose>0.0 0.0 -0.06533 0.0 0.0 0.0</pose>
+      <axis>
+        <xyz>0 1 0</xyz>
+        <limit>
+          <lower>-0.785</lower>
+          <upper>0.785</upper>
+        </limit>
+        <dynamics>
+          <friction>0</friction>
+          <damping>10</damping>
+        </dynamics>
+      </axis>
+    </joint>
+  </gazebo>
+  <gazebo>
+    <joint name="differential_right_pin_parallel_joint"
+           type="revolute" >
+      <parent>differential_right_pin_link</parent>
+      <child>right_side_link</child>
+      <pose>0.0 0.0 -0.06533 0.0 0.0 0.0</pose>
+      <axis>
+        <xyz>0 1 0</xyz>
+        <limit>
+          <lower>-0.785</lower>
+          <upper>0.785</upper>
+        </limit>
+        <dynamics>
+          <friction>0</friction>
+          <damping>10</damping>
+        </dynamics>
+      </axis>
+    </joint>
+  </gazebo>
   <gazebo reference="left_front_wheel_link" >
     <minDepth>${wheel_min_depth}</minDepth>

Commit message: Rename picam sensor name

File: pandora_gazebo_description/gio/urdf_gazebo/gio.gazebo.xacro (robot description, xacro)
@@ -15,13 +15,14 @@
     <xacro:kinect_sensor />
   </xacro:if>
+  <xacro:if value="${enable_picam}" >
+    <xacro:picam_sensor prefix="front" />
+    <xacro:picam_sensor prefix="rear" />
+  </xacro:if>
+  <xacro:if value="${enable_webcam}" >
+    <xacro:webcam_sensor prefix="left" />
+    <xacro:webcam_sensor prefix="right" />
+  </xacro:if>
   <xacro:if value="${enable_thermal}" >
     <xacro:thermal_sensor />
-  </xacro:if>
-  <xacro:if value="${enable_camera_effector}" >
-    <xacro:camera_effector_sensor />
-  </xacro:if>
-  <xacro:if value="${enable_webcam}" >
-    <xacro:webcam_sensor prefix_y="left" />
-    <xacro:webcam_sensor prefix_y="right" />
   </xacro:if>
   <xacro:if value="${enable_sonar}" >

File: pandora_gazebo_description/gio/urdf_gazebo/sdf_configurations.xacro (robot description, xacro)
@@ -6,7 +6,7 @@
   <xacro:property name="enable_laser" value="true" />
   <xacro:property name="enable_kinect" value="true" />
+  <xacro:property name="enable_picam" value="true" />
+  <xacro:property name="enable_webcam" value="true" />
   <xacro:property name="enable_thermal" value="false" />
-  <xacro:property name="enable_camera_effector" value="true" />
-  <xacro:property name="enable_webcam" value="true" />
   <xacro:property name="enable_sonar" value="true" />
   <xacro:property name="enable_co2" value="true" />

File: pandora_gazebo_description/sdf_elements/sensors/picam.gazebo.xacro (robot description, xacro)
@@ -1,7 +1,7 @@
 <?xml version="1.0"?>
 <robot xmlns:xacro="http://ros.org/wiki/xacro" >
-  <xacro:macro name="camera_effector_sensor" >
-    <gazebo reference="pi_camera_frame" >
-      <sensor name="pi_camera" type="camera" >
+  <xacro:macro name="picam_sensor" params="prefix" >
+    <gazebo reference="${prefix}_picam_frame" >
+      <sensor name="${prefix}_picam" type="camera" >
         <camera>
           <horizontal_fov>0.93375114982</horizontal_fov>

File: pandora_gazebo_description/sdf_elements/sensors/webcam.gazebo.xacro (robot description, xacro)
@@ -1,9 +1,9 @@
 <?xml version="1.0"?>
 <robot xmlns:xacro="http://ros.org/wiki/xacro" >
-  <xacro:macro name="webcam_sensor" params="prefix_y" >
-    <gazebo reference="${prefix_y}_camera_frame" >
-      <sensor name="${prefix_y}_camera" type="camera" >
+  <xacro:macro name="webcam_sensor" params="prefix" >
+    <gazebo reference="${prefix}_webcam_frame" >
+      <sensor name="${prefix}_webcam" type="camera" >
         <camera>
-          <horizontal_fov>1.047197551</horizontal_fov>
+          <horizontal_fov>1.06465084</horizontal_fov>
           <image>
             <width>1280</width>
@@ -17,6 +17,6 @@
         </camera>
         <plugin name="camera2ros" filename="libgazebo_ros_camera.so" >
-          <frameName>${prefix_y}_camera_optical_frame</frameName>
-          <cameraName>${prefix_y}_camera</cameraName>
+          <frameName>${prefix}_webcam_optical_frame</frameName>
+          <cameraName>${prefix}_camera</cameraName>
           <imageTopicName>image</imageTopicName>
         </plugin>

Commit message: Add secondary picam macro

File: pandora_gazebo_description/gio/urdf_gazebo/gio.gazebo.xacro (robot description, xacro)
@@ -16,6 +16,6 @@
   </xacro:if>
   <xacro:if value="${enable_picam}" >
-    <xacro:picam_sensor prefix="front" />
-    <xacro:picam_sensor prefix="rear" />
+    <xacro:front_picam_sensor />
+    <xacro:rear_picam_sensor />
   </xacro:if>
   <xacro:if value="${enable_webcam}" >

File: pandora_gazebo_description/sdf_elements/sensors/picam.gazebo.xacro (robot description, xacro)
@@ -1,9 +1,9 @@
 <?xml version="1.0"?>
 <robot xmlns:xacro="http://ros.org/wiki/xacro" >
-  <xacro:macro name="picam_sensor" params="prefix" >
-    <gazebo reference="${prefix}_picam_frame" >
-      <sensor name="${prefix}_picam" type="camera" >
+  <xacro:macro name="front_picam_sensor" >
+    <gazebo reference="front_picam_frame" >
+      <sensor name="front_picam" type="camera" >
         <camera>
-          <horizontal_fov>0.93375114982</horizontal_fov>
+          <horizontal_fov>0.93375115</horizontal_fov>
           <image>
             <width>640</width>
@@ -17,6 +17,32 @@
         </camera>
         <plugin name="camera2ros" filename="libgazebo_ros_camera.so" >
-          <frameName>pi_camera_optical_frame</frameName>
-          <cameraName>rpi2/pi_camera</cameraName>
+          <frameName>front_picam_optical_frame</frameName>
+          <cameraName>rpi2_primary/pi_camera_front</cameraName>
+          <imageTopicName>image</imageTopicName>
+        </plugin>
+        <always_on>1</always_on>
+        <update_rate>5</update_rate>
+        <visualize>false</visualize>
+      </sensor>
+    </gazebo>
+  </xacro:macro>
+  <xacro:macro name="rear_picam_sensor" >
+    <gazebo reference="rear_picam_frame" >
+      <sensor name="rear_picam" type="camera" >
+        <camera>
+          <horizontal_fov>0.93375115</horizontal_fov>
+          <image>
+            <width>1280</width>
+            <height>720</height>
+            <format>R8G8B8</format>
+          </image>
+          <clip>
+            <near>0.15</near>
+            <far>2.0</far>
+          </clip>
+        </camera>
+        <plugin name="camera2ros" filename="libgazebo_ros_camera.so" >
+          <frameName>rear_picam_optical_frame</frameName>
+          <cameraName>rpi2_secondary/pi_camera_rear</cameraName>
           <imageTopicName>image</imageTopicName>
         </plugin>

Commit message: Disable physical differential joint, add plugin instead

File: pandora_gazebo_description/gio/urdf_gazebo/gio.gazebo.xacro (robot description, xacro)
@@ -38,4 +38,6 @@
   <!-- Load Plugins -->
   <xacro:gazebo_ros_control interface="pandora_gazebo_interface/GioGazeboInterface" />
+  <xacro:pandora_differential />
+  <!--<xacro:ros_skid_steer_drive />-->
   <xacro:pandora_p3d />
   <xacro:if value="$(arg tune)" >

File: pandora_gazebo_description/gio/urdf_gazebo/references.gazebo.xacro (robot description, xacro)
@@ -1,42 +1,42 @@
 <?xml version="1.0" ?>
 <robot xmlns:xacro="http://ros.org/wiki/xacro" >
-  <gazebo>
-    <joint name="differential_left_pin_parallel_joint"
-           type="revolute" >
-      <parent>differential_left_pin_link</parent>
-      <child>left_side_link</child>
-      <pose>0.0 0.0 -0.06533 0.0 0.0 0.0</pose>
-      <axis>
-        <xyz>0 1 0</xyz>
-        <limit>
-          <lower>-0.785</lower>
-          <upper>0.785</upper>
-        </limit>
-        <dynamics>
-          <friction>0</friction>
-          <damping>10</damping>
-        </dynamics>
-      </axis>
-    </joint>
-  </gazebo>
-  <gazebo>
-    <joint name="differential_right_pin_parallel_joint"
-           type="revolute" >
-      <parent>differential_right_pin_link</parent>
-      <child>right_side_link</child>
-      <pose>0.0 0.0 -0.06533 0.0 0.0 0.0</pose>
-      <axis>
-        <xyz>0 1 0</xyz>
-        <limit>
-          <lower>-0.785</lower>
-          <upper>0.785</upper>
-        </limit>
-        <dynamics>
-          <friction>0</friction>
-          <damping>10</damping>
-        </dynamics>
-      </axis>
-    </joint>
-  </gazebo>
+  <!--<gazebo>-->
+    <!--<joint name="differential_left_pin_parallel_joint"-->
+           <!--type="revolute" >-->
+      <!--<parent>differential_left_pin_link</parent>-->
+      <!--<child>left_side_link</child>-->
+      <!--<pose>0.0 0.0 -0.06533 0.0 0.0 0.0</pose>-->
+      <!--<axis>-->
+        <!--<xyz>0 1 0</xyz>-->
+        <!--<limit>-->
+          <!--<lower>-0.785</lower>-->
+          <!--<upper>0.785</upper>-->
+        <!--</limit>-->
+        <!--<dynamics>-->
+          <!--<friction>0</friction>-->
+          <!--<damping>10</damping>-->
+        <!--</dynamics>-->
+      <!--</axis>-->
+    <!--</joint>-->
+  <!--</gazebo>-->
+  <!--<gazebo>-->
+    <!--<joint name="differential_right_pin_parallel_joint"-->
+           <!--type="revolute" >-->
+      <!--<parent>differential_right_pin_link</parent>-->
+      <!--<child>right_side_link</child>-->
+      <!--<pose>0.0 0.0 -0.06533 0.0 0.0 0.0</pose>-->
+      <!--<axis>-->
+        <!--<xyz>0 1 0</xyz>-->
+        <!--<limit>-->
+          <!--<lower>-0.785</lower>-->
+          <!--<upper>0.785</upper>-->
+        <!--</limit>-->
+        <!--<dynamics>-->
+          <!--<friction>0</friction>-->
+          <!--<damping>10</damping>-->
+        <!--</dynamics>-->
+      <!--</axis>-->
+    <!--</joint>-->
+  <!--</gazebo>-->
   <gazebo reference="linear_actuator_joint" >
     <implicitSpringDamper>true</implicitSpringDamper>

File: pandora_gazebo_description/sdf_elements/sensors/kinect.gazebo.xacro (robot description, xacro)
@@ -24,4 +24,5 @@
           <depthImageCameraInfoTopicName>depth/image/info</depthImageCameraInfoTopicName>
           <pointCloudCutoff>0.4</pointCloudCutoff>
+          <pointCloudCutoffMax>5</pointCloudCutoffMax>
         </plugin>
         <always_on>1</always_on>

Commit message: Changes in sensors, friction
* Add gpu enabled laser sensor, able of update rates more than 5Hz
* Enable ROS imu plugin, publishes velocities, acceleration, covariance
* Change params on kinect sensor

File: pandora_gazebo_description/gio/urdf_gazebo/gio.gazebo.xacro (robot description, xacro)
@@ -10,5 +10,6 @@
   <!-- Load gazebo sensors -->
   <xacro:if value="${enable_laser}" >
-    <xacro:laser_sensor range="${laser_range}" />
+    <!--<xacro:laser_sensor range="${laser_range}" update_rate="${laser_update_rate}" />-->
+    <xacro:laser_sensor_gpu range="${laser_range}" update_rate="${laser_update_rate}" />
   </xacro:if>
   <xacro:if value="${enable_kinect}" >
@@ -39,4 +40,5 @@
   <xacro:gazebo_ros_control interface="pandora_gazebo_interface/GioGazeboInterface" />
   <xacro:pandora_differential />
+  <xacro:ros_imu />
   <!--<xacro:ros_skid_steer_drive />-->
   <xacro:pandora_p3d />

File: pandora_gazebo_description/gio/urdf_gazebo/sdf_configurations.xacro (robot description, xacro)
@@ -3,4 +3,5 @@
   <!-- Sensor properties -->
   <xacro:property name="laser_range" value="20" />
+  <xacro:property name="laser_update_rate" value="10" />
   <!-- Enable gazebo sensors -->
   <xacro:property name="enable_laser" value="true" />
@@ -13,6 +14,6 @@
   <xacro:property name="enable_microphone" value="false" />
   <!-- Wheel physics -->
-  <xacro:property name="wheel_mu_1" value="0.85" />
-  <xacro:property name="wheel_mu_2" value="0.70" />
+  <xacro:property name="wheel_mu_1" value="0.7" />
+  <xacro:property name="wheel_mu_2" value="0.7" />
   <xacro:property name="wheel_k_p" value="1000000.0" />
   <xacro:property name="wheel_k_d" value="1.0" />

File: pandora_gazebo_description/sdf_elements/plugins/ros_imu_plugin.gazebo.xacro (robot description, xacro)
@@ -5,5 +5,5 @@
       <plugin name="RosImuPlugin" filename="libgazebo_ros_imu.so" >
         <updateRate>50.0</updateRate>
-        <topicName>/sensors/imu</topicName>
+        <topicName>/sensors/imu_all</topicName>
         <serviceName>default_imu</serviceName>
         <robotNamespace>/</robotNamespace>

File: pandora_gazebo_description/sdf_elements/sensors/kinect.gazebo.xacro (robot description, xacro)
@@ -5,5 +5,6 @@
       <sensor name="kinect" type="depth" >
         <camera>
-          <horizontal_fov>1.012290966</horizontal_fov>
+          <!--<horizontal_fov>1.012290966</horizontal_fov>-->
+          <horizontal_fov>1.57</horizontal_fov>
           <image>
             <width>640</width>
@@ -12,6 +13,6 @@
           </image>
           <clip>
-            <near>0.3</near>
-            <far>3</far>
+            <near>0.2</near>
+            <far>7</far>
           </clip>
         </camera>
@@ -23,6 +24,6 @@
           <depthImageTopicName>depth/image</depthImageTopicName>
           <depthImageCameraInfoTopicName>depth/image/info</depthImageCameraInfoTopicName>
-          <pointCloudCutoff>0.4</pointCloudCutoff>
-          <pointCloudCutoffMax>5</pointCloudCutoffMax>
+          <pointCloudCutoff>0.2</pointCloudCutoff>
+          <pointCloudCutoffMax>7</pointCloudCutoffMax>
         </plugin>
         <always_on>1</always_on>

File: pandora_gazebo_description/sdf_elements/sensors/laser.gazebo.xacro (robot description, xacro)
@@ -1,7 +1,10 @@
 <?xml version="1.0"?>
 <robot xmlns:xacro="http://ros.org/wiki/xacro" >
-  <xacro:macro name="laser_sensor" params="range" >
+  <xacro:macro name="laser_sensor" params="range update_rate" >
     <gazebo reference="laser_link" >
       <sensor name="laser" type="ray" >
+        <always_on>true</always_on>
+        <update_rate>${update_rate}</update_rate>
+        <visualize>true</visualize>
         <ray>
           <scan>
@@ -18,13 +21,47 @@
             <resolution>0.01</resolution>
           </range>
+          <noise>
+            <type>gaussian</type>
+            <mean>0.0</mean>
+            <stddev>0.001</stddev>
+          </noise>
         </ray>
-        <plugin name="laser" filename="libRayPlugin.so" />
         <plugin name="laser2Ros" filename="libgazebo_ros_laser.so" >
           <frameName>/laser_link</frameName>
           <topicName>/laser/scan</topicName>
         </plugin>
-        <always_on>1</always_on>
-        <update_rate>10</update_rate>
+      </sensor>
+    </gazebo>
+  </xacro:macro>
+  <xacro:macro name="laser_sensor_gpu" params="range update_rate" >
+    <gazebo reference="laser_link" >
+      <sensor name="laser" type="gpu_ray" >
+        <always_on>true</always_on>
+        <update_rate>${update_rate}</update_rate>
         <visualize>true</visualize>
+        <ray>
+          <scan>
+            <horizontal>
+              <samples>683</samples>
+              <resolution>1</resolution>
+              <min_angle>-2.00712864</min_angle>
+              <max_angle>2.00712864</max_angle>
+            </horizontal>
+          </scan>
+          <range>
+            <min>0.08</min>
+            <max>${range}</max>
+            <resolution>0.01</resolution>
+          </range>
+          <noise>
+            <type>gaussian</type>
+            <mean>0.0</mean>
+            <stddev>0.001</stddev>
+          </noise>
+        </ray>
+        <plugin name="laser2Ros" filename="libgazebo_ros_gpu_laser.so" >
+          <frameName>/laser_link</frameName>
+          <topicName>/laser/scan</topicName>
+        </plugin>
       </sensor>
     </gazebo>
