Commit message: Remove picam sensor from monstertruck description

File: pandora_gazebo_description/monstertruck/urdf_gazebo/monstertruck.gazebo.xacro (robot description, xacro)
@@ -12,7 +12,4 @@
     <xacro:laser_sensor_gpu range="${laser_range}" update_rate="${laser_update_rate}" />
   </xacro:if>
-  <xacro:if value="${enable_picam}" >
-    <xacro:front_picam_sensor />
-  </xacro:if>
   <!-- Load Plugins -->
   <xacro:gazebo_ros_control interface="pandora_gazebo_interface/MonstertruckGazeboInterface" />

File: pandora_gazebo_description/monstertruck/urdf_gazebo/sdf_configurations.xacro (robot description, xacro)
@@ -6,5 +6,4 @@
   <!-- Enable gazebo sensors -->
   <xacro:property name="enable_laser" value="true" />
-  <xacro:property name="enable_picam" value="true" />
   <!-- Calibrate Wheel physics TODO(gkouros) -->
   <xacro:property name="wheel_mu_1" value="0.7" />
