Commit message: Adjust monstertruck parameters

File: pandora_gazebo_description/monstertruck/urdf_gazebo/sdf_configurations.xacro (robot description, xacro)
@@ -7,6 +7,6 @@
   <xacro:property name="enable_laser" value="true" />
   <!-- Calibrate Wheel physics TODO(gkouros) -->
-  <xacro:property name="wheel_mu_1" value="0.7" />
-  <xacro:property name="wheel_mu_2" value="0.7" />
+  <xacro:property name="wheel_mu_1" value="0.5" />
+  <xacro:property name="wheel_mu_2" value="0.5" />
   <xacro:property name="wheel_k_p" value="1000000.0" />
   <xacro:property name="wheel_k_d" value="1.0" />
